File: clock.kicad_sch (KiCad schematic)
At the start: 8 parts, among them U17 74HC74, U9 74HCU04, Y1 3.58Mhz

Commit message: Update to KiCad v10 and use plugin-based Artemisa libs
Parts:
- C20, C36, C37: footprint artemisa:Disc_capacitor -> PCM_artemisa:Disc_capacitor; symbol artemisa:Cap -> PCM_artemisa:Cap
- R23, R24: footprint artemisa:Axial_resistor -> PCM_artemisa:Axial_resistor; symbol artemisa:R -> PCM_artemisa:R
- U17: footprint artemisa:DIP-14_300 -> PCM_artemisa:DIP-14_300; symbol artemisa:74HC74 -> PCM_artemisa:74HC74
- U9: footprint artemisa:DIP-14_300 -> PCM_artemisa:DIP-14_300; symbol artemisa:74HCU04 -> PCM_artemisa:74HCU04
- Y1: footprint artemisa:Crystal -> PCM_artemisa:Crystal; symbol artemisa:Crystal -> PCM_artemisa:Crystal
