File: cpu.kicad_sch (KiCad schematic)
At the start: 12 parts, among them U3 74HCT244, U4 74HCT244, U5 74HCT244, U6 Z84C00, U7 74HC74, U8 74HCT245

Commit message: Update to KiCad v10 and use plugin-based Artemisa libs
Parts:
- C15, C16, C17, C19, C3, C4: footprint artemisa:Disc_capacitor -> PCM_artemisa:Disc_capacitor; symbol artemisa:Cap -> PCM_artemisa:Cap
- U3, U4, U5: footprint artemisa:DIP-20_300 -> PCM_artemisa:DIP-20_300; symbol artemisa:74HCT244 -> PCM_artemisa:74HCT244
- U6: footprint artemisa:DIP-40_600 -> PCM_artemisa:DIP-40_600; symbol artemisa:Z84C00 -> PCM_artemisa:Z84C00
- U7: footprint artemisa:DIP-14_300 -> PCM_artemisa:DIP-14_300; symbol artemisa:74HC74 -> PCM_artemisa:74HC74
- U8: footprint artemisa:DIP-20_300 -> PCM_artemisa:DIP-20_300; symbol artemisa:74HCT245 -> PCM_artemisa:74HCT245
