File: cpu.kicad_sch (KiCad schematic)
At the start: 12 parts, among them U3 74HCT244, U4 74HCT244, U5 74HCT244, U6 Z84C00, U7 74HC74, U8 74HCT245

Commit message: Re-annotate the whole schematic
Parts:
- renumbered C17 to C10, C3 to C11, C4 to C12, C15 to C7, C19 to C8, C16 to C9, U7 to U10, U4 to U11, U5 to U12, U6 to U13, U8 to U14, U3 to U9

Commit message: Adjust footprints and draft PCB layout
Parts:
- C10, C11, C12, C7, C8, C9: footprint PCM_artemisa:Disc_capacitor -> Capacitor_THT:C_Disc_D5.0mm_W2.5mm_P2.50mm
- U10: footprint PCM_artemisa:DIP-14_300 -> Package_DIP:DIP-14_W7.62mm
- U11, U12, U14, U9: footprint PCM_artemisa:DIP-20_300 -> Package_DIP:DIP-20_W7.62mm
- U13: footprint PCM_artemisa:DIP-40_600 -> Package_DIP:DIP-40_W15.24mm_Socket
Changed lines of the file:
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@@
 			)
 		)
-		(property "Footprint" "PCM_artemisa:DIP-40_600"
+		(property "Footprint" "Package_DIP:DIP-40_W15.24mm_Socket"
 			(at 148.59 97.79 0)
 			(hide yes)
@@
 			)
 		)
-		(property "Footprint" "PCM_artemisa:DIP-20_300"
+		(property "Footprint" "Package_DIP:DIP-20_W7.62mm"
 			(at 210.82 35.56 0)
 			(hide yes)
@@
 			)
 		)
-		(property "Footprint" "PCM_artemisa:DIP-20_300"
+		(property "Footprint" "Package_DIP:DIP-20_W7.62mm"
 			(at 210.82 59.69 0)
 			(hide yes)
@@
 			)
 		)
-		(property "Footprint" "PCM_artemisa:DIP-20_300"
+		(property "Footprint" "Package_DIP:DIP-20_W7.62mm"
 			(at 210.82 83.82 0)
 			(hide yes)
@@
 			)
 		)
-		(property "Footprint" "PCM_artemisa:DIP-20_300"
+		(property "Footprint" "Package_DIP:DIP-20_W7.62mm"
 			(at 210.82 107.95 0)
 			(hide yes)
@@
 			)
 		)
-		(property "Footprint" "PCM_artemisa:DIP-20_300"
+		(property "Footprint" "Package_DIP:DIP-20_W7.62mm"
 			(at 210.82 152.4 0)
 			(hide yes)
@@
 			)
 		)
-		(property "Footprint" "PCM_artemisa:DIP-20_300"
+		(property "Footprint" "Package_DIP:DIP-20_W7.62mm"
 			(at 74.93 60.96 0)
 			(hide yes)
@@
 			)
 		)
-		(property "Footprint" "PCM_artemisa:DIP-20_300"
+		(property "Footprint" "Package_DIP:DIP-20_W7.62mm"
 			(at 74.93 90.17 0)
 			(hide yes)
@@
 			)
 		)
-		(property "Footprint" "PCM_artemisa:DIP-14_300"
+		(property "Footprint" "Package_DIP:DIP-14_W7.62mm"
 			(at 69.85 146.05 0)
 			(hide yes)
@@
 			)
 		)
-		(property "Footprint" "PCM_artemisa:DIP-14_300"
+		(property "Footprint" "Package_DIP:DIP-14_W7.62mm"
 			(at 111.76 146.05 0)
 			(hide yes)
@@
 			)
 		)
-		(property "Footprint" "PCM_artemisa:Disc_capacitor"
+		(property "Footprint" "Capacitor_THT:C_Disc_D5.0mm_W2.5mm_P2.50mm"
 			(at 215.9 116.84 0)
 			(hide yes)
@@
 			)
 		)
-		(property "Footprint" "PCM_artemisa:Disc_capacitor"
+		(property "Footprint" "Capacitor_THT:C_Disc_D5.0mm_W2.5mm_P2.50mm"
 			(at 156.21 53.34 0)
 			(hide yes)
@@
 			)
 		)
-		(property "Footprint" "PCM_artemisa:DIP-20_300"
+		(property "Footprint" "Package_DIP:DIP-20_W7.62mm"
 			(at 50.8 191.77 0)
 			(hide yes)
@@
 			)
 		)
-		(property "Footprint" "PCM_artemisa:Disc_capacitor"
+		(property "Footprint" "Capacitor_THT:C_Disc_D5.0mm_W2.5mm_P2.50mm"
 			(at 58.42 181.61 0)
 			(hide yes)
@@
 			)
 		)
-		(property "Footprint" "PCM_artemisa:DIP-20_300"
+		(property "Footprint" "Package_DIP:DIP-20_W7.62mm"
 			(at 76.2 191.77 0)
 			(hide yes)
@@
 			)
 		)
-		(property "Footprint" "PCM_artemisa:Disc_capacitor"
+		(property "Footprint" "Capacitor_THT:C_Disc_D5.0mm_W2.5mm_P2.50mm"
 			(at 83.82 181.61 0)
 			(hide yes)
@@
 			)
 		)
-		(property "Footprint" "PCM_artemisa:DIP-20_300"
+		(property "Footprint" "Package_DIP:DIP-20_W7.62mm"
 			(at 101.6 191.77 0)
 			(hide yes)
@@
 			)
 		)
-		(property "Footprint" "PCM_artemisa:Disc_capacitor"
+		(property "Footprint" "Capacitor_THT:C_Disc_D5.0mm_W2.5mm_P2.50mm"
 			(at 109.22 181.61 0)
 			(hide yes)
@@
 			)
 		)
-		(property "Footprint" "PCM_artemisa:Disc_capacitor"
+		(property "Footprint" "Capacitor_THT:C_Disc_D5.0mm_W2.5mm_P2.50mm"
 			(at 77.47 125.73 0)
 			(hide yes)
