File: decoding.kicad_sch (KiCad schematic)
At the start: 14 parts, among them U10 74HC04, U11 74HC32, U12 74HC32, U13 74HC32, U14 74HC08, U15 74HC139, U17 74HC74, U26 74HC138

Commit message: Update to KiCad v10 and use plugin-based Artemisa libs
Parts:
- C10, C11, C12, C13, C38, C8: footprint artemisa:Disc_capacitor -> PCM_artemisa:Disc_capacitor; symbol artemisa:Cap -> PCM_artemisa:Cap
- U10: footprint artemisa:DIP-14_300 -> PCM_artemisa:DIP-14_300; symbol artemisa:74HC04 -> PCM_artemisa:74HC04
- U11, U12, U13: footprint artemisa:DIP-14_300 -> PCM_artemisa:DIP-14_300; symbol artemisa:74HC32 -> PCM_artemisa:74HC32
- U14: footprint artemisa:DIP-14_300 -> PCM_artemisa:DIP-14_300; symbol artemisa:74HC08 -> PCM_artemisa:74HC08
- U15: footprint artemisa:DIP-16_300 -> PCM_artemisa:DIP-16_300; symbol artemisa:74HC139 -> PCM_artemisa:74HC139
- U17: footprint artemisa:DIP-14_300 -> PCM_artemisa:DIP-14_300; symbol artemisa:74HC74 -> PCM_artemisa:74HC74
- U26: footprint artemisa:DIP-16_300 -> PCM_artemisa:DIP-16_300; symbol artemisa:74HC138 -> PCM_artemisa:74HC138
