File: decoding.kicad_sch (KiCad schematic)
At the start: 14 parts, among them U10 74HC04, U11 74HC32, U12 74HC32, U13 74HC32, U14 74HC08, U15 74HC139, U17 74HC74, U26 74HC138

Commit message: Re-annotate the whole schematic
Parts:
- renumbered C8 to C1, C12 to C2, C11 to C3, C13 to C4, C38 to C5, C10 to C6, U10 to U1, U13 to U2, U11 to U3, U12 to U4, U15 to U5, U14 to U6, U26 to U7, U17 to U8

Commit message: Adjust footprints and draft PCB layout
Parts:
- C1, C2, C3, C4, C5, C6: footprint PCM_artemisa:Disc_capacitor -> Capacitor_THT:C_Disc_D5.0mm_W2.5mm_P2.50mm
- U1, U2, U3, U4, U6, U8: footprint PCM_artemisa:DIP-14_300 -> Package_DIP:DIP-14_W7.62mm
- U5, U7: footprint PCM_artemisa:DIP-16_300 -> Package_DIP:DIP-16_W7.62mm
Changed lines of the file:
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@@
 			)
 		)
-		(property "Footprint" "PCM_artemisa:DIP-14_300"
+		(property "Footprint" "Package_DIP:DIP-14_W7.62mm"
 			(at 101.6 222.25 0)
 			(hide yes)
@@
 			)
 		)
-		(property "Footprint" "PCM_artemisa:DIP-14_300"
+		(property "Footprint" "Package_DIP:DIP-14_W7.62mm"
 			(at 134.62 243.84 0)
 			(hide yes)
@@
 			)
 		)
-		(property "Footprint" "PCM_artemisa:DIP-14_300"
+		(property "Footprint" "Package_DIP:DIP-14_W7.62mm"
 			(at 101.6 234.95 0)
 			(hide yes)
@@
 			)
 		)
-		(property "Footprint" "PCM_artemisa:DIP-14_300"
+		(property "Footprint" "Package_DIP:DIP-14_W7.62mm"
 			(at 134.62 213.36 0)
 			(hide yes)
@@
 			)
 		)
-		(property "Footprint" "PCM_artemisa:DIP-14_300"
+		(property "Footprint" "Package_DIP:DIP-14_W7.62mm"
 			(at 184.15 204.47 0)
 			(hide yes)
@@
 			)
 		)
-		(property "Footprint" "PCM_artemisa:DIP-14_300"
+		(property "Footprint" "Package_DIP:DIP-14_W7.62mm"
 			(at 161.29 215.9 0)
 			(hide yes)
@@
 			)
 		)
-		(property "Footprint" "PCM_artemisa:DIP-14_300"
+		(property "Footprint" "Package_DIP:DIP-14_W7.62mm"
 			(at 205.74 204.47 0)
 			(hide yes)
@@
 			)
 		)
-		(property "Footprint" "PCM_artemisa:DIP-14_300"
+		(property "Footprint" "Package_DIP:DIP-14_W7.62mm"
 			(at 205.74 243.84 0)
 			(hide yes)
@@
 			)
 		)
-		(property "Footprint" "PCM_artemisa:DIP-14_300"
+		(property "Footprint" "Package_DIP:DIP-14_W7.62mm"
 			(at 99.06 210.82 0)
 			(hide yes)
@@
 			)
 		)
-		(property "Footprint" "PCM_artemisa:DIP-14_300"
+		(property "Footprint" "Package_DIP:DIP-14_W7.62mm"
 			(at 165.1 67.31 0)
 			(hide yes)
@@
 			)
 		)
-		(property "Footprint" "PCM_artemisa:DIP-14_300"
+		(property "Footprint" "Package_DIP:DIP-14_W7.62mm"
 			(at 137.16 78.74 0)
 			(hide yes)
@@
 			)
 		)
-		(property "Footprint" "PCM_artemisa:DIP-14_300"
+		(property "Footprint" "Package_DIP:DIP-14_W7.62mm"
 			(at 137.16 102.87 0)
 			(hide yes)
@@
 			)
 		)
-		(property "Footprint" "PCM_artemisa:DIP-14_300"
+		(property "Footprint" "Package_DIP:DIP-14_W7.62mm"
 			(at 137.16 115.57 0)
 			(hide yes)
@@
 			)
 		)
-		(property "Footprint" "PCM_artemisa:DIP-16_300"
+		(property "Footprint" "Package_DIP:DIP-16_W7.62mm"
 			(at 137.16 138.43 0)
 			(hide yes)
@@
 			)
 		)
-		(property "Footprint" "PCM_artemisa:DIP-14_300"
+		(property "Footprint" "Package_DIP:DIP-14_W7.62mm"
 			(at 165.1 134.62 0)
 			(hide yes)
@@
 			)
 		)
-		(property "Footprint" "PCM_artemisa:DIP-16_300"
+		(property "Footprint" "Package_DIP:DIP-16_W7.62mm"
 			(at 153.67 276.86 90)
 			(hide yes)
@@
 			)
 		)
-		(property "Footprint" "PCM_artemisa:DIP-14_300"
+		(property "Footprint" "Package_DIP:DIP-14_W7.62mm"
 			(at 92.71 295.91 0)
 			(hide yes)
@@
 			)
 		)
-		(property "Footprint" "PCM_artemisa:DIP-14_300"
+		(property "Footprint" "Package_DIP:DIP-14_W7.62mm"
 			(at 113.03 298.45 0)
 			(hide yes)
@@
 			)
 		)
-		(property "Footprint" "PCM_artemisa:DIP-14_300"
+		(property "Footprint" "Package_DIP:DIP-14_W7.62mm"
 			(at 134.62 154.94 0)
 			(hide yes)
@@
 			)
 		)
-		(property "Footprint" "PCM_artemisa:DIP-14_300"
+		(property "Footprint" "Package_DIP:DIP-14_W7.62mm"
 			(at 158.75 152.4 0)
 			(hide yes)
@@
 			)
 		)
-		(property "Footprint" "PCM_artemisa:DIP-14_300"
+		(property "Footprint" "Package_DIP:DIP-14_W7.62mm"
 			(at 184.15 170.18 0)
 			(hide yes)
@@
 			)
 		)
-		(property "Footprint" "PCM_artemisa:DIP-14_300"
+		(property "Footprint" "Package_DIP:DIP-14_W7.62mm"
 			(at 184.15 187.96 0)
 			(hide yes)
@@
 			)
 		)
-		(property "Footprint" "PCM_artemisa:DIP-14_300"
+		(property "Footprint" "Package_DIP:DIP-14_W7.62mm"
 			(at 95.25 190.5 0)
 			(hide yes)
@@
 			)
 		)
-		(property "Footprint" "PCM_artemisa:DIP-14_300"
+		(property "Footprint" "Package_DIP:DIP-14_W7.62mm"
 			(at 181.61 335.28 0)
 			(hide yes)
@@
 			)
 		)
-		(property "Footprint" "PCM_artemisa:Disc_capacitor"
+		(property "Footprint" "Capacitor_THT:C_Disc_D5.0mm_W2.5mm_P2.50mm"
 			(at 182.88 257.81 0)
 			(hide yes)
@@
 			)
 		)
-		(property "Footprint" "PCM_artemisa:Disc_capacitor"
+		(property "Footprint" "Capacitor_THT:C_Disc_D5.0mm_W2.5mm_P2.50mm"
 			(at 107.95 182.88 0)
 			(hide yes)
@@
 			)
 		)
-		(property "Footprint" "PCM_artemisa:Disc_capacitor"
+		(property "Footprint" "Capacitor_THT:C_Disc_D5.0mm_W2.5mm_P2.50mm"
 			(at 130.81 66.04 0)
 			(hide yes)
@@
 			)
 		)
-		(property "Footprint" "PCM_artemisa:Disc_capacitor"
+		(property "Footprint" "Capacitor_THT:C_Disc_D5.0mm_W2.5mm_P2.50mm"
 			(at 129.54 288.29 0)
 			(hide yes)
@@
 			)
 		)
-		(property "Footprint" "PCM_artemisa:Disc_capacitor"
+		(property "Footprint" "Capacitor_THT:C_Disc_D5.0mm_W2.5mm_P2.50mm"
 			(at 173.99 54.61 0)
 			(hide yes)
@@
 			)
 		)
-		(property "Footprint" "PCM_artemisa:Disc_capacitor"
+		(property "Footprint" "Capacitor_THT:C_Disc_D5.0mm_W2.5mm_P2.50mm"
 			(at 195.58 160.02 0)
 			(hide yes)
