File: keyboard.kicad_sch (KiCad schematic)
At the start: 8 parts, among them J2 DB25M, U16 74LS07, U21 74HC138, U22 74HC138

Commit message: Update to KiCad v10 and use plugin-based Artemisa libs
Parts:
- C18, C24, C25: footprint artemisa:Disc_capacitor -> PCM_artemisa:Disc_capacitor; symbol artemisa:Cap -> PCM_artemisa:Cap
- J2: footprint artemisa:DB25M -> PCM_artemisa:DB25M; symbol artemisa:DB25M -> PCM_artemisa:DB25M
- RN2: footprint artemisa:RN8 -> PCM_artemisa:RN8; symbol artemisa:RN8 -> PCM_artemisa:RN8
- U16: footprint artemisa:DIP-14_300 -> PCM_artemisa:DIP-14_300; symbol artemisa:74LS07 -> PCM_artemisa:74LS07
- U21, U22: footprint artemisa:DIP-16_300 -> PCM_artemisa:DIP-16_300; symbol artemisa:74HC138 -> PCM_artemisa:74HC138
