File: keyboard.kicad_sch (KiCad schematic)
At the start: 8 parts, among them J2 DB25M, U16 74LS07, U21 74HC138, U22 74HC138

Commit message: Re-annotate the whole schematic
Parts:
- renumbered C24 to C16, C25 to C17, J2 to J1, RN2 to RN1, U16 to U17, U21 to U18, U22 to U19
Changed lines of the file:
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@@
 		(in_pos_files yes)
 		(dnp no)
-		(property "Reference" "RN2"
+		(property "Reference" "RN1"
 			(at 103.632 24.0538 0)
 			(show_name no)
@@
 			(project "motherboard-hk10"
 				(path "/e63e39d7-6ac0-4ffd-8aa3-1841a4541b55/00000000-0000-0000-0000-00005ae5dd12"
-					(reference "RN2")
+					(reference "RN1")
 					(unit 1)
 				)
@@
 		(in_pos_files yes)
 		(dnp no)
-		(property "Reference" "J2"
+		(property "Reference" "J1"
 			(at 201.3712 79.4004 0)
 			(show_name no)
@@
 			(project "motherboard-hk10"
 				(path "/e63e39d7-6ac0-4ffd-8aa3-1841a4541b55/00000000-0000-0000-0000-00005ae5dd12"
-					(reference "J2")
+					(reference "J1")
 					(unit 1)
 				)
@@
 		(in_pos_files yes)
 		(dnp no)
-		(property "Reference" "#PWR068"
+		(property "Reference" "#PWR064"
 			(at 193.04 46.99 0)
 			(hide yes)
@@
 			(project "motherboard-hk10"
 				(path "/e63e39d7-6ac0-4ffd-8aa3-1841a4541b55/00000000-0000-0000-0000-00005ae5dd12"
-					(reference "#PWR068")
+					(reference "#PWR064")
 					(unit 1)
 				)
@@
 		(in_pos_files yes)
 		(dnp no)
-		(property "Reference" "#PWR076"
+		(property "Reference" "#PWR065"
 			(at 193.04 115.57 0)
 			(hide yes)
@@
 			(project "motherboard-hk10"
 				(path "/e63e39d7-6ac0-4ffd-8aa3-1841a4541b55/00000000-0000-0000-0000-00005ae5dd12"
-					(reference "#PWR076")
+					(reference "#PWR065")
 					(unit 1)
 				)
@@
 		(in_pos_files yes)
 		(dnp no)
-		(property "Reference" "#PWR067"
+		(property "Reference" "#PWR057"
 			(at 114.3 19.05 0)
 			(hide yes)
@@
 			(project "motherboard-hk10"
 				(path "/e63e39d7-6ac0-4ffd-8aa3-1841a4541b55/00000000-0000-0000-0000-00005ae5dd12"
-					(reference "#PWR067")
+					(reference "#PWR057")
 					(unit 1)
 				)
@@
 		(in_pos_files yes)
 		(dnp no)
-		(property "Reference" "U16"
+		(property "Reference" "U17"
 			(at 110.49 130.81 0)
 			(show_name no)
@@
 			(project "motherboard-hk10"
 				(path "/e63e39d7-6ac0-4ffd-8aa3-1841a4541b55/00000000-0000-0000-0000-00005ae5dd12"
-					(reference "U16")
+					(reference "U17")
 					(unit 5)
 				)
@@
 		(in_pos_files yes)
 		(dnp no)
-		(property "Reference" "U16"
+		(property "Reference" "U17"
 			(at 110.49 138.43 0)
 			(show_name no)
@@
 			(project "motherboard-hk10"
 				(path "/e63e39d7-6ac0-4ffd-8aa3-1841a4541b55/00000000-0000-0000-0000-00005ae5dd12"
-					(reference "U16")
+					(reference "U17")
 					(unit 6)
 				)
@@
 		(in_pos_files yes)
 		(dnp no)
-		(property "Reference" "U21"
+		(property "Reference" "U18"
 			(at 129.54 54.61 0)
 			(show_name no)
@@
 			(project "motherboard-hk10"
 				(path "/e63e39d7-6ac0-4ffd-8aa3-1841a4541b55/00000000-0000-0000-0000-00005ae5dd12"
-					(reference "U21")
+					(reference "U18")
 					(unit 1)
 				)
@@
 		(in_pos_files yes)
 		(dnp no)
-		(property "Reference" "U22"
+		(property "Reference" "U19"
 			(at 129.54 95.25 0)
 			(show_name no)
@@
 			(project "motherboard-hk10"
 				(path "/e63e39d7-6ac0-4ffd-8aa3-1841a4541b55/00000000-0000-0000-0000-00005ae5dd12"
-					(reference "U22")
+					(reference "U19")
 					(unit 1)
 				)
@@
 		(in_pos_files yes)
 		(dnp no)
-		(property "Reference" "#PWR073"
+		(property "Reference" "#PWR059"
 			(at 137.16 83.82 0)
 			(hide yes)
@@
 			(project "motherboard-hk10"
 				(path "/e63e39d7-6ac0-4ffd-8aa3-1841a4541b55/00000000-0000-0000-0000-00005ae5dd12"
-					(reference "#PWR073")
+					(reference "#PWR059")
 					(unit 1)
 				)
@@
 		(in_pos_files yes)
 		(dnp no)
-		(property "Reference" "#PWR074"
+		(property "Reference" "#PWR060"
 			(at 137.16 90.17 0)
 			(hide yes)
@@
 			(project "motherboard-hk10"
 				(path "/e63e39d7-6ac0-4ffd-8aa3-1841a4541b55/00000000-0000-0000-0000-00005ae5dd12"
-					(reference "#PWR074")
+					(reference "#PWR060")
 					(unit 1)
 				)
@@
 		(in_pos_files yes)
 		(dnp no)
-		(property "Reference" "C25"
+		(property "Reference" "C17"
 			(at 143.51 90.17 90)
 			(show_name no)
@@
 			(project "motherboard-hk10"
 				(path "/e63e39d7-6ac0-4ffd-8aa3-1841a4541b55/00000000-0000-0000-0000-00005ae5dd12"
-					(reference "C25")
+					(reference "C17")
 					(unit 1)
 				)
@@
 		(in_pos_files yes)
 		(dnp no)
-		(property "Reference" "#PWR075"
+		(property "Reference" "#PWR063"
 			(at 149.86 96.52 0)
 			(hide yes)
@@
 			(project "motherboard-hk10"
 				(path "/e63e39d7-6ac0-4ffd-8aa3-1841a4541b55/00000000-0000-0000-0000-00005ae5dd12"
-					(reference "#PWR075")
+					(reference "#PWR063")
 					(unit 1)
 				)
@@
 		(in_pos_files yes)
 		(dnp no)
-		(property "Reference" "#PWR072"
+		(property "Reference" "#PWR054"
 			(at 110.49 81.28 0)
 			(hide yes)
@@
 			(project "motherboard-hk10"
 				(path "/e63e39d7-6ac0-4ffd-8aa3-1841a4541b55/00000000-0000-0000-0000-00005ae5dd12"
-					(reference "#PWR072")
+					(reference "#PWR054")
 					(unit 1)
 				)
@@
 		(in_pos_files yes)
 		(dnp no)
-		(property "Reference" "#PWR071"
+		(property "Reference" "#PWR056"
 			(at 113.03 69.85 0)
 			(hide yes)
@@
 			(project "motherboard-hk10"
 				(path "/e63e39d7-6ac0-4ffd-8aa3-1841a4541b55/00000000-0000-0000-0000-00005ae5dd12"
-					(reference "#PWR071")
+					(reference "#PWR056")
 					(unit 1)
 				)
@@
 		(in_pos_files yes)
 		(dnp no)
-		(property "Reference" "#PWR077"
+		(property "Reference" "#PWR055"
 			(at 110.49 121.92 0)
 			(hide yes)
@@
 			(project "motherboard-hk10"
 				(path "/e63e39d7-6ac0-4ffd-8aa3-1841a4541b55/00000000-0000-0000-0000-00005ae5dd12"
-					(reference "#PWR077")
+					(reference "#PWR055")
 					(unit 1)
 				)
@@
 		(in_pos_files yes)
 		(dnp no)
-		(property "Reference" "#PWR069"
+		(property "Reference" "#PWR058"
 			(at 137.16 49.53 0)
 			(hide yes)
@@
 			(project "motherboard-hk10"
 				(path "/e63e39d7-6ac0-4ffd-8aa3-1841a4541b55/00000000-0000-0000-0000-00005ae5dd12"
-					(reference "#PWR069")
+					(reference "#PWR058")
 					(unit 1)
 				)
@@
 		(in_pos_files yes)
 		(dnp no)
-		(property "Reference" "C24"
+		(property "Reference" "C16"
 			(at 143.51 49.53 90)
 			(show_name no)
@@
 			(project "motherboard-hk10"
 				(path "/e63e39d7-6ac0-4ffd-8aa3-1841a4541b55/00000000-0000-0000-0000-00005ae5dd12"
-					(reference "C24")
+					(reference "C16")
 					(unit 1)
 				)
@@
 		(in_pos_files yes)
 		(dnp no)
-		(property "Reference" "#PWR070"
+		(property "Reference" "#PWR062"
 			(at 149.86 55.88 0)
 			(hide yes)
@@
 			(project "motherboard-hk10"
 				(path "/e63e39d7-6ac0-4ffd-8aa3-1841a4541b55/00000000-0000-0000-0000-00005ae5dd12"
-					(reference "#PWR070")
+					(reference "#PWR062")
 					(unit 1)
 				)
@@
 		(in_pos_files yes)
 		(dnp no)
-		(property "Reference" "#PWR078"
+		(property "Reference" "#PWR061"
 			(at 137.16 124.46 0)
 			(hide yes)
@@
 			(project "motherboard-hk10"
 				(path "/e63e39d7-6ac0-4ffd-8aa3-1841a4541b55/00000000-0000-0000-0000-00005ae5dd12"
-					(reference "#PWR078")
+					(reference "#PWR061")
 					(unit 1)
 				)
@@
 		(in_pos_files yes)
 		(dnp no)
-		(property "Reference" "U16"
+		(property "Reference" "U17"
 			(at 236.22 50.8 90)
 			(show_name no)
@@
 			(project "motherboard-hk10"
 				(path "/e63e39d7-6ac0-4ffd-8aa3-1841a4541b55/00000000-0000-0000-0000-00005ae5dd12"
-					(reference "U16")
+					(reference "U17")
 					(unit 7)
 				)
@@
 		(in_pos_files yes)
 		(dnp no)
-		(property "Reference" "#PWR0158"
+		(property "Reference" "#PWR067"
 			(at 241.3 68.58 0)
 			(hide yes)
@@
 			(project "motherboard-hk10"
 				(path "/e63e39d7-6ac0-4ffd-8aa3-1841a4541b55/00000000-0000-0000-0000-00005ae5dd12"
-					(reference "#PWR0158")
+					(reference "#PWR067")
 					(unit 1)
 				)
@@
 		(in_pos_files yes)
 		(dnp no)
-		(property "Reference" "#PWR0159"
+		(property "Reference" "#PWR066"
 			(at 241.3 46.99 0)
 			(hide yes)
@@
 			(project "motherboard-hk10"
 				(path "/e63e39d7-6ac0-4ffd-8aa3-1841a4541b55/00000000-0000-0000-0000-00005ae5dd12"
-					(reference "#PWR0159")
+					(reference "#PWR066")
 					(unit 1)
 				)

Commit message: Adjust footprints and draft PCB layout
Parts:
- C16, C17, C18: footprint PCM_artemisa:Disc_capacitor -> Capacitor_THT:C_Disc_D5.0mm_W2.5mm_P2.50mm
- RN1: footprint PCM_artemisa:RN8 -> Resistor_THT:R_Array_SIP9
- U17: footprint PCM_artemisa:DIP-14_300 -> Package_DIP:DIP-14_W7.62mm
- U18, U19: footprint PCM_artemisa:DIP-16_300 -> Package_DIP:DIP-16_W7.62mm
Changed lines of the file:
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@@
 			)
 		)
-		(property "Footprint" "PCM_artemisa:RN8"
+		(property "Footprint" "Resistor_THT:R_Array_SIP9"
 			(at 121.92 28.575 0)
 			(hide yes)
@@
 			)
 		)
-		(property "Footprint" "PCM_artemisa:DIP-14_300"
+		(property "Footprint" "Package_DIP:DIP-14_W7.62mm"
 			(at 115.57 134.62 0)
 			(hide yes)
@@
 			)
 		)
-		(property "Footprint" "PCM_artemisa:DIP-14_300"
+		(property "Footprint" "Package_DIP:DIP-14_W7.62mm"
 			(at 115.57 142.24 0)
 			(hide yes)
@@
 			)
 		)
-		(property "Footprint" "PCM_artemisa:DIP-16_300"
+		(property "Footprint" "Package_DIP:DIP-16_W7.62mm"
 			(at 115.57 69.85 90)
 			(hide yes)
@@
 			)
 		)
-		(property "Footprint" "PCM_artemisa:DIP-16_300"
+		(property "Footprint" "Package_DIP:DIP-16_W7.62mm"
 			(at 115.57 110.49 90)
 			(hide yes)
@@
 			)
 		)
-		(property "Footprint" "PCM_artemisa:Disc_capacitor"
+		(property "Footprint" "Capacitor_THT:C_Disc_D5.0mm_W2.5mm_P2.50mm"
 			(at 144.78 91.44 0)
 			(hide yes)
@@
 			)
 		)
-		(property "Footprint" "PCM_artemisa:Disc_capacitor"
+		(property "Footprint" "Capacitor_THT:C_Disc_D5.0mm_W2.5mm_P2.50mm"
 			(at 144.78 50.8 0)
 			(hide yes)
@@
 			)
 		)
-		(property "Footprint" "PCM_artemisa:DIP-14_300"
+		(property "Footprint" "Package_DIP:DIP-14_W7.62mm"
 			(at 241.3 55.88 0)
 			(hide yes)
@@
 			)
 		)
-		(property "Footprint" "PCM_artemisa:Disc_capacitor"
+		(property "Footprint" "Capacitor_THT:C_Disc_D5.0mm_W2.5mm_P2.50mm"
 			(at 248.92 55.88 0)
 			(hide yes)
