File: motherboard-101.kicad_sch (KiCad schematic)
At the start: 0 parts

Commit message: Update to KiCad v10 and use plugin-based Artemisa libs
Other:
- sheet CPU ports: added none; removed ~{VDPINT}
- sheet SLOTS ports: added ~{EXTINT}; removed ~{EXITINT}
