File: power.kicad_sch (KiCad schematic)
At the start: 16 parts, among them J1 PWR_conn, Q1 2N2222, SW1 Push_button, U9 74HCU04

Commit message: Update to KiCad v10 and use plugin-based Artemisa libs
Parts:
- C5, C6, C7: footprint artemisa:Radial_capacitor -> PCM_artemisa:Radial_capacitor; symbol artemisa:CP -> PCM_artemisa:CP
- C9: footprint artemisa:Disc_capacitor -> PCM_artemisa:Disc_capacitor; symbol artemisa:Cap -> PCM_artemisa:Cap
- D1: footprint artemisa:Axial_diode -> PCM_artemisa:Axial_diode; symbol artemisa:1N4448 -> PCM_artemisa:1N4448
- D2: footprint artemisa:LED -> PCM_artemisa:LED; symbol artemisa:LED -> PCM_artemisa:LED
- J1: footprint artemisa:Jack_55_21 -> PCM_artemisa:Jack_55_21; symbol artemisa:PWR_conn -> PCM_artemisa:PWR_conn
- Q1: footprint artemisa:TO92 -> PCM_artemisa:TO92; symbol artemisa:2N2222 -> PCM_artemisa:2N2222
- R1, R2, R3, R4, R5, R6: footprint artemisa:Axial_resistor -> PCM_artemisa:Axial_resistor; symbol artemisa:R -> PCM_artemisa:R
- SW1: footprint artemisa:Push_button_angled -> PCM_artemisa:Push_button_angled; symbol artemisa:Push_button -> PCM_artemisa:Push_button
- U9: footprint artemisa:DIP-14_300 -> PCM_artemisa:DIP-14_300; symbol artemisa:74HCU04 -> PCM_artemisa:74HCU04
