File: ppi.kicad_sch (KiCad schematic)
At the start: 6 parts, among them U15 74HC139, U27 74HC153, U28 82C55A

Commit message: Update to KiCad v10 and use plugin-based Artemisa libs
Parts:
- C14, C39, C40: footprint artemisa:Disc_capacitor -> PCM_artemisa:Disc_capacitor; symbol artemisa:Cap -> PCM_artemisa:Cap
- U15: footprint artemisa:DIP-16_300 -> PCM_artemisa:DIP-16_300; symbol artemisa:74HC139 -> PCM_artemisa:74HC139
- U27: footprint artemisa:DIP-16_300 -> PCM_artemisa:DIP-16_300; symbol artemisa:74HC153 -> PCM_artemisa:74HC153
- U28: footprint artemisa:DIP-40_600 -> PCM_artemisa:DIP-40_600; symbol artemisa:82C55A -> PCM_artemisa:82C55A
