File: psg.kicad_sch (KiCad schematic)
At the start: 21 parts, among them J6 CONN_JOY, J7 CONN_JOY, U14 74HC08, U16 74LS07, U23 74HC157, U24 AY-3-8910, U25 74HC157

Commit message: Update to KiCad v10 and use plugin-based Artemisa libs
Parts:
- C26, C27, C28: footprint artemisa:Disc_capacitor -> PCM_artemisa:Disc_capacitor; symbol artemisa:Cap -> PCM_artemisa:Cap
- C29, C30, C31: footprint artemisa:Radial_capacitor -> PCM_artemisa:Radial_capacitor; symbol artemisa:CP -> PCM_artemisa:CP
- J6, J7: footprint artemisa:Joystick_conn -> PCM_artemisa:Joystick_conn; symbol artemisa:CONN_JOY -> PCM_artemisa:CONN_JOY
- R10, R11, R12, R7, R8, R9: footprint artemisa:Axial_resistor -> PCM_artemisa:Axial_resistor; symbol artemisa:R -> PCM_artemisa:R
- RN4: footprint artemisa:RN8 -> PCM_artemisa:RN8; symbol artemisa:RN8 -> PCM_artemisa:RN8
- RN5: footprint artemisa:RN4 -> PCM_artemisa:RN4; symbol artemisa:RN4 -> PCM_artemisa:RN4
- U14: footprint artemisa:DIP-14_300 -> PCM_artemisa:DIP-14_300; symbol artemisa:74HC08 -> PCM_artemisa:74HC08
- U16: footprint artemisa:DIP-14_300 -> PCM_artemisa:DIP-14_300; symbol artemisa:74LS07 -> PCM_artemisa:74LS07
- U23, U25: footprint artemisa:DIP-16_300 -> PCM_artemisa:DIP-16_300; symbol artemisa:74HC157 -> PCM_artemisa:74HC157
- U24: footprint artemisa:DIP-40_600 -> PCM_artemisa:DIP-40_600; symbol artemisa:AY-3-8910 -> PCM_artemisa:AY-3-8910
