File: psg.kicad_sch (KiCad schematic)
At the start: 21 parts, among them J6 CONN_JOY, J7 CONN_JOY, U14 74HC08, U16 74LS07, U23 74HC157, U24 AY-3-8910, U25 74HC157

Commit message: Use clock generator IC instead of oscillator
Parts:
- removed U14: 74HC08, PCM_artemisa:DIP-14_300, symbol PCM_artemisa:74HC08
Connections:
- no-connect marks 5 -> 4
Changed lines of the file:
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@@
 	)
 	(junction
-		(at 213.36 193.04)
-		(diameter 0)
-		(color 0 0 0 0)
-	)
-	(junction
 		(at 260.35 52.07)
 		(diameter 0)
@@
 	)
 	(no_connect
-		(at 240.03 190.5)
-	)
-	(no_connect
 		(at 214.63 90.17)
 	)
@@
 		)
 	)
-	(wire
-		(pts
-			(xy 213.36 187.96) (xy 213.36 193.04)
-		)
-		(stroke
-			(width 0)
-			(type default)
-		)
-	)
 	(bus
 		(pts
@@
 	(wire
 		(pts
-			(xy 213.36 193.04) (xy 213.36 198.12)
-		)
-		(stroke
-			(width 0)
-			(type default)
-		)
-	)
-	(wire
-		(pts
 			(xy 144.78 184.15) (xy 144.78 189.23)
 		)
@@
 	(wire
 		(pts
-			(xy 218.44 187.96) (xy 213.36 187.96)
-		)
-		(stroke
-			(width 0)
-			(type default)
-		)
-	)
-	(wire
-		(pts
 			(xy 113.03 69.85) (xy 121.92 69.85)
 		)
@@
 	(wire
 		(pts
-			(xy 218.44 193.04) (xy 213.36 193.04)
-		)
-		(stroke
-			(width 0)
-			(type default)
-		)
-	)
-	(wire
-		(pts
 			(xy 152.4 109.22) (xy 152.4 165.1)
 		)
@@
 					(unit 1)
 				)
-			)
-		)
-	)
-	(symbol
-		(lib_id "PCM_artemisa:74HC08")
-		(at 229.87 190.5 0)
-		(unit 4)
-		(body_style 2)
-		(exclude_from_sim no)
-		(in_bom yes)
-		(on_board yes)
-		(in_pos_files yes)
-		(dnp no)
-		(property "Reference" "U14"
-			(at 229.87 185.42 0)
-			(show_name no)
-			(do_not_autoplace no)
-			(effects
-				(font
-					(size 1.27 1.27)
-				)
-			)
-		)
-		(property "Value" "74HC08"
-			(at 229.87 195.58 0)
-			(show_name no)
-			(do_not_autoplace no)
-			(effects
-				(font
-					(size 1.27 1.27)
-				)
-			)
-		)
-		(property "Footprint" "PCM_artemisa:DIP-14_300"
-			(at 229.87 190.5 0)
-			(hide yes)
-			(show_name no)
-			(do_not_autoplace no)
-			(effects
-				(font
-					(size 1.27 1.27)
-				)
-			)
-		)
-		(property "Datasheet" ""
-			(at 229.87 190.5 0)
-			(hide yes)
-			(show_name no)
-			(do_not_autoplace no)
-			(effects
-				(font
-					(size 1.27 1.27)
-				)
-			)
-		)
-		(property "Description" ""
-			(at 229.87 190.5 0)
-			(hide yes)
-			(show_name no)
-			(do_not_autoplace no)
-			(effects
-				(font
-					(size 1.27 1.27)
-				)
-			)
-		)
-		(pin "14"
-		)
-		(pin "7"
-		)
-		(pin "1"
-		)
-		(pin "2"
-		)
-		(pin "3"
-		)
-		(pin "4"
-		)
-		(pin "5"
-		)
-		(pin "6"
-		)
-		(pin "10"
-		)
-		(pin "8"
-		)
-		(pin "9"
-		)
-		(pin "11"
-		)
-		(pin "12"
-		)
-		(pin "13"
-		)
-		(instances
-			(project "motherboard-hk10"
-				(path "/e63e39d7-6ac0-4ffd-8aa3-1841a4541b55/00000000-0000-0000-0000-00005aed18cc"
-					(reference "U14")
-					(unit 4)
-				)
-			)
-		)
-	)
-	(symbol
-		(lib_id "PCM_artemisa:GND")
-		(at 213.36 198.12 0)
-		(unit 1)
-		(body_style 1)
-		(exclude_from_sim no)
-		(in_bom yes)
-		(on_board yes)
-		(in_pos_files yes)
-		(dnp no)
-		(property "Reference" "#PWR0115"
-			(at 213.36 200.66 0)
-			(hide yes)
-			(show_name no)
-			(do_not_autoplace no)
-			(effects
-				(font
-					(size 1.524 1.524)
-				)
-			)
-		)
-		(property "Value" "GND"
-			(at 213.36 195.58 0)
-			(hide yes)
-			(show_name no)
-			(do_not_autoplace no)
-			(effects
-				(font
-					(size 1.524 1.524)
-				)
-			)
-		)
-		(property "Footprint" ""
-			(at 213.36 198.12 0)
-			(hide yes)
-			(show_name no)
-			(do_not_autoplace no)
-			(effects
-				(font
-					(size 1.524 1.524)
-				)
-			)
-		)
-		(property "Datasheet" ""
-			(at 213.36 198.12 0)
-			(hide yes)
-			(show_name no)
-			(do_not_autoplace no)
-			(effects
-				(font
-					(size 1.524 1.524)
-				)
-			)
-		)
-		(property "Description" ""
-			(at 213.36 198.12 0)
-			(hide yes)
-			(show_name no)
-			(do_not_autoplace no)
-			(effects
-				(font
-					(size 1.27 1.27)
-				)
-			)
-		)
-		(pin ""
-		)
-		(instances
-			(project "motherboard-hk10"
-				(path "/e63e39d7-6ac0-4ffd-8aa3-1841a4541b55/00000000-0000-0000-0000-00005aed18cc"
-					(reference "#PWR0115")
-					(unit 1)
-				)

Commit message: Re-annotate the whole schematic
Parts:
- renumbered C29 to C32, C30 to C33, C27 to C34, C31 to C35, C26 to C36, C28 to C37, R10 to R3, R11 to R4, R12 to R5, R8 to R6, R9 to R7, R7 to R8, U16 to U17, U24 to U25, U23 to U26, U25 to U27

Commit message: Adjust footprints and draft PCB layout
Parts:
- C32, C33, C35: footprint PCM_artemisa:Radial_capacitor -> Capacitor_THT:CP_Radial_D4.0mm_P2.00mm
- C34, C36, C37: footprint PCM_artemisa:Disc_capacitor -> Capacitor_THT:C_Disc_D5.0mm_W2.5mm_P2.50mm
- R3, R4, R5, R6, R7, R8: footprint PCM_artemisa:Axial_resistor -> Resistor_THT:R_Axial_DIN0207_L6.3mm_D2.5mm_P10.16mm_Horizontal
- RN4: footprint PCM_artemisa:RN8 -> Resistor_THT:R_Array_SIP9
- RN5: footprint PCM_artemisa:RN4 -> Resistor_THT:R_Array_SIP5
- U17: footprint PCM_artemisa:DIP-14_300 -> Package_DIP:DIP-14_W7.62mm
- U25: footprint PCM_artemisa:DIP-40_600 -> Package_DIP:DIP-40_W15.24mm_Socket
- U26, U27: footprint PCM_artemisa:DIP-16_300 -> Package_DIP:DIP-16_W7.62mm
Changed lines of the file:
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@@
 			)
 		)
-		(property "Footprint" "PCM_artemisa:DIP-40_600"
+		(property "Footprint" "Package_DIP:DIP-40_W15.24mm_Socket"
 			(at 137.16 83.82 0)
 			(hide yes)
@@
 			)
 		)
-		(property "Footprint" "PCM_artemisa:DIP-16_300"
+		(property "Footprint" "Package_DIP:DIP-16_W7.62mm"
 			(at 227.33 68.58 0)
 			(hide yes)
@@
 			)
 		)
-		(property "Footprint" "PCM_artemisa:DIP-16_300"
+		(property "Footprint" "Package_DIP:DIP-16_W7.62mm"
 			(at 227.33 106.68 0)
 			(hide yes)
@@
 			)
 		)
-		(property "Footprint" "PCM_artemisa:DIP-14_300"
+		(property "Footprint" "Package_DIP:DIP-14_W7.62mm"
 			(at 227.33 119.38 0)
 			(hide yes)
@@
 			)
 		)
-		(property "Footprint" "PCM_artemisa:DIP-14_300"
+		(property "Footprint" "Package_DIP:DIP-14_W7.62mm"
 			(at 227.33 128.27 0)
 			(hide yes)
@@
 			)
 		)
-		(property "Footprint" "PCM_artemisa:DIP-14_300"
+		(property "Footprint" "Package_DIP:DIP-14_W7.62mm"
 			(at 227.33 137.16 0)
 			(hide yes)
@@
 			)
 		)
-		(property "Footprint" "PCM_artemisa:DIP-14_300"
+		(property "Footprint" "Package_DIP:DIP-14_W7.62mm"
 			(at 227.33 146.05 0)
 			(hide yes)
@@
 			)
 		)
-		(property "Footprint" "PCM_artemisa:Axial_resistor"
+		(property "Footprint" "Resistor_THT:R_Axial_DIN0207_L6.3mm_D2.5mm_P10.16mm_Horizontal"
 			(at 156.21 113.792 90)
 			(hide yes)
@@
 			)
 		)
-		(property "Footprint" "PCM_artemisa:Radial_capacitor"
+		(property "Footprint" "Capacitor_THT:CP_Radial_D4.0mm_P2.00mm"
 			(at 152.4 167.64 0)
 			(hide yes)
@@
 			)
 		)
-		(property "Footprint" "PCM_artemisa:Axial_resistor"
+		(property "Footprint" "Resistor_THT:R_Axial_DIN0207_L6.3mm_D2.5mm_P10.16mm_Horizontal"
 			(at 152.4 178.562 90)
 			(hide yes)
@@
 			)
 		)
-		(property "Footprint" "PCM_artemisa:Radial_capacitor"
+		(property "Footprint" "Capacitor_THT:CP_Radial_D4.0mm_P2.00mm"
 			(at 137.16 167.64 0)
 			(hide yes)
@@
 			)
 		)
-		(property "Footprint" "PCM_artemisa:Axial_resistor"
+		(property "Footprint" "Resistor_THT:R_Axial_DIN0207_L6.3mm_D2.5mm_P10.16mm_Horizontal"
 			(at 137.16 178.562 90)
 			(hide yes)
@@
 			)
 		)
-		(property "Footprint" "PCM_artemisa:Radial_capacitor"
+		(property "Footprint" "Capacitor_THT:CP_Radial_D4.0mm_P2.00mm"
 			(at 144.78 167.64 0)
 			(hide yes)
@@
 			)
 		)
-		(property "Footprint" "PCM_artemisa:Axial_resistor"
+		(property "Footprint" "Resistor_THT:R_Axial_DIN0207_L6.3mm_D2.5mm_P10.16mm_Horizontal"
 			(at 144.78 178.562 90)
 			(hide yes)
@@
 			)
 		)
-		(property "Footprint" "PCM_artemisa:Axial_resistor"
+		(property "Footprint" "Resistor_THT:R_Axial_DIN0207_L6.3mm_D2.5mm_P10.16mm_Horizontal"
 			(at 162.56 113.792 90)
 			(hide yes)
@@
 			)
 		)
-		(property "Footprint" "PCM_artemisa:Axial_resistor"
+		(property "Footprint" "Resistor_THT:R_Axial_DIN0207_L6.3mm_D2.5mm_P10.16mm_Horizontal"
 			(at 168.91 45.212 90)
 			(hide yes)
@@
 			)
 		)
-		(property "Footprint" "PCM_artemisa:RN8"
+		(property "Footprint" "Resistor_THT:R_Array_SIP9"
 			(at 251.46 34.925 0)
 			(hide yes)
@@
 			)
 		)
-		(property "Footprint" "PCM_artemisa:RN4"
+		(property "Footprint" "Resistor_THT:R_Array_SIP5"
 			(at 259.715 76.2 0)
 			(hide yes)
@@
 			)
 		)
-		(property "Footprint" "PCM_artemisa:Disc_capacitor"
+		(property "Footprint" "Capacitor_THT:C_Disc_D5.0mm_W2.5mm_P2.50mm"
 			(at 146.05 45.72 0)
 			(hide yes)
@@
 			)
 		)
-		(property "Footprint" "PCM_artemisa:Disc_capacitor"
+		(property "Footprint" "Capacitor_THT:C_Disc_D5.0mm_W2.5mm_P2.50mm"
 			(at 236.22 35.56 0)
 			(hide yes)
@@
 			)
 		)
-		(property "Footprint" "PCM_artemisa:Disc_capacitor"
+		(property "Footprint" "Capacitor_THT:C_Disc_D5.0mm_W2.5mm_P2.50mm"
 			(at 236.22 74.93 0)
 			(hide yes)
