File: ram.kicad_sch (KiCad schematic)
At the start: 4 parts, among them U1 62256, U2 62256

Commit message: Update to KiCad v10 and use plugin-based Artemisa libs
Parts:
- C1, C2: footprint artemisa:Disc_capacitor -> PCM_artemisa:Disc_capacitor; symbol artemisa:Cap -> PCM_artemisa:Cap
- U1, U2: footprint artemisa:DIP-28_600 -> PCM_artemisa:DIP-28_600; symbol artemisa:62256 -> PCM_artemisa:62256
