File: ram.kicad_sch (KiCad schematic)
At the start: 4 parts, among them U1 62256, U2 62256

Commit message: Re-annotate the whole schematic
Parts:
- renumbered C1 to C29, C2 to C30, U1 to U22, U2 to U23
Changed lines of the file:
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@@
 		(in_pos_files yes)
 		(dnp no)
-		(property "Reference" "U1"
+		(property "Reference" "U22"
 			(at 119.38 55.88 0)
 			(show_name no)
@@
 			(project "motherboard-hk10"
 				(path "/e63e39d7-6ac0-4ffd-8aa3-1841a4541b55/00000000-0000-0000-0000-00005ad4d0ed"
-					(reference "U1")
+					(reference "U22")
 					(unit 1)
 				)
@@
 		(in_pos_files yes)
 		(dnp no)
-		(property "Reference" "U2"
+		(property "Reference" "U23"
 			(at 198.12 55.88 0)
 			(show_name no)
@@
 			(project "motherboard-hk10"
 				(path "/e63e39d7-6ac0-4ffd-8aa3-1841a4541b55/00000000-0000-0000-0000-00005ad4d0ed"
-					(reference "U2")
+					(reference "U23")
 					(unit 1)
 				)
@@
 		(in_pos_files yes)
 		(dnp no)
-		(property "Reference" "#PWR05"
+		(property "Reference" "#PWR094"
 			(at 128.27 102.87 0)
 			(hide yes)
@@
 			(project "motherboard-hk10"
 				(path "/e63e39d7-6ac0-4ffd-8aa3-1841a4541b55/00000000-0000-0000-0000-00005ad4d0ed"
-					(reference "#PWR05")
+					(reference "#PWR094")
 					(unit 1)
 				)
@@
 		(in_pos_files yes)
 		(dnp no)
-		(property "Reference" "#PWR06"
+		(property "Reference" "#PWR097"
 			(at 207.01 102.87 0)
 			(hide yes)
@@
 			(project "motherboard-hk10"
 				(path "/e63e39d7-6ac0-4ffd-8aa3-1841a4541b55/00000000-0000-0000-0000-00005ad4d0ed"
-					(reference "#PWR06")
+					(reference "#PWR097")
 					(unit 1)
 				)
@@
 		(in_pos_files yes)
 		(dnp no)
-		(property "Reference" "#PWR01"
+		(property "Reference" "#PWR093"
 			(at 128.27 45.72 0)
 			(hide yes)
@@
 			(project "motherboard-hk10"
 				(path "/e63e39d7-6ac0-4ffd-8aa3-1841a4541b55/00000000-0000-0000-0000-00005ad4d0ed"
-					(reference "#PWR01")
+					(reference "#PWR093")
 					(unit 1)
 				)
@@
 		(in_pos_files yes)
 		(dnp no)
-		(property "Reference" "C1"
+		(property "Reference" "C29"
 			(at 133.35 46.99 90)
 			(show_name no)
@@
 			(project "motherboard-hk10"
 				(path "/e63e39d7-6ac0-4ffd-8aa3-1841a4541b55/00000000-0000-0000-0000-00005ad4d0ed"
-					(reference "C1")
+					(reference "C29")
 					(unit 1)
 				)
@@
 		(in_pos_files yes)
 		(dnp no)
-		(property "Reference" "#PWR03"
+		(property "Reference" "#PWR095"
 			(at 139.7 53.34 0)
 			(hide yes)
@@
 			(project "motherboard-hk10"
 				(path "/e63e39d7-6ac0-4ffd-8aa3-1841a4541b55/00000000-0000-0000-0000-00005ad4d0ed"
-					(reference "#PWR03")
+					(reference "#PWR095")
 					(unit 1)
 				)
@@
 		(in_pos_files yes)
 		(dnp no)
-		(property "Reference" "#PWR02"
+		(property "Reference" "#PWR096"
 			(at 207.01 45.72 0)
 			(hide yes)
@@
 			(project "motherboard-hk10"
 				(path "/e63e39d7-6ac0-4ffd-8aa3-1841a4541b55/00000000-0000-0000-0000-00005ad4d0ed"
-					(reference "#PWR02")
+					(reference "#PWR096")
 					(unit 1)
 				)
@@
 		(in_pos_files yes)
 		(dnp no)
-		(property "Reference" "C2"
+		(property "Reference" "C30"
 			(at 212.09 46.99 90)
 			(show_name no)
@@
 			(project "motherboard-hk10"
 				(path "/e63e39d7-6ac0-4ffd-8aa3-1841a4541b55/00000000-0000-0000-0000-00005ad4d0ed"
-					(reference "C2")
+					(reference "C30")
 					(unit 1)
 				)
@@
 		(in_pos_files yes)
 		(dnp no)
-		(property "Reference" "#PWR04"
+		(property "Reference" "#PWR098"
 			(at 218.44 53.34 0)
 			(hide yes)
@@
 			(project "motherboard-hk10"
 				(path "/e63e39d7-6ac0-4ffd-8aa3-1841a4541b55/00000000-0000-0000-0000-00005ad4d0ed"
-					(reference "#PWR04")
-					(unit 1)
-				)
+					(reference "#PWR098")
+					(unit 1)
+				)

Commit message: Adjust footprints and draft PCB layout
Parts:
- C29, C30: footprint PCM_artemisa:Disc_capacitor -> Capacitor_THT:C_Disc_D5.0mm_W2.5mm_P2.50mm
- U22, U23: footprint PCM_artemisa:DIP-28_600 -> Package_DIP:DIP-28_W15.24mm_Socket
Changed lines of the file:
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@@
 			)
 		)
-		(property "Footprint" "PCM_artemisa:DIP-28_600"
+		(property "Footprint" "Package_DIP:DIP-28_W15.24mm_Socket"
 			(at 128.27 81.28 0)
 			(hide yes)
@@
 			)
 		)
-		(property "Footprint" "PCM_artemisa:DIP-28_600"
+		(property "Footprint" "Package_DIP:DIP-28_W15.24mm_Socket"
 			(at 207.01 81.28 0)
 			(hide yes)
@@
 			)
 		)
-		(property "Footprint" "PCM_artemisa:Disc_capacitor"
+		(property "Footprint" "Capacitor_THT:C_Disc_D5.0mm_W2.5mm_P2.50mm"
 			(at 134.62 48.26 0)
 			(hide yes)
@@
 			)
 		)
-		(property "Footprint" "PCM_artemisa:Disc_capacitor"
+		(property "Footprint" "Capacitor_THT:C_Disc_D5.0mm_W2.5mm_P2.50mm"
 			(at 213.36 48.26 0)
 			(hide yes)
