File: rom.kicad_sch (KiCad schematic)
At the start: 7 parts, among them U20 SST39SF0

Commit message: Update to KiCad v10 and use plugin-based Artemisa libs
Parts:
- C23: footprint artemisa:Disc_capacitor -> PCM_artemisa:Disc_capacitor; symbol artemisa:Cap -> PCM_artemisa:Cap
- JP1, JP2, JP3, JP4: footprint artemisa:Jumper -> PCM_artemisa:Jumper; symbol artemisa:Jumper -> PCM_artemisa:Jumper
- RN1: footprint artemisa:RN4 -> PCM_artemisa:RN4; symbol artemisa:RN4 -> PCM_artemisa:RN4
- U20: footprint artemisa:DIP-32_600 -> PCM_artemisa:DIP-32_600; symbol artemisa:SST39SF0 -> PCM_artemisa:SST39SF0
