File: rom.kicad_sch (KiCad schematic)
At the start: 7 parts, among them U20 SST39SF0

Commit message: Re-annotate the whole schematic
Parts:
- renumbered C23 to C28, RN1 to RN2, U20 to U21
Changed lines of the file:
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@@
 		(in_pos_files yes)
 		(dnp no)
-		(property "Reference" "U20"
+		(property "Reference" "U21"
 			(at 133.35 48.26 0)
 			(show_name no)
@@
 			(project "motherboard-hk10"
 				(path "/e63e39d7-6ac0-4ffd-8aa3-1841a4541b55/00000000-0000-0000-0000-00005ae56078"
-					(reference "U20")
+					(reference "U21")
 					(unit 1)
 				)
@@
 		(in_pos_files yes)
 		(dnp no)
-		(property "Reference" "#PWR062"
+		(property "Reference" "#PWR092"
 			(at 161.29 78.74 0)
 			(hide yes)
@@
 			(project "motherboard-hk10"
 				(path "/e63e39d7-6ac0-4ffd-8aa3-1841a4541b55/00000000-0000-0000-0000-00005ae56078"
-					(reference "#PWR062")
+					(reference "#PWR092")
 					(unit 1)
 				)
@@
 		(in_pos_files yes)
 		(dnp no)
-		(property "Reference" "RN1"
+		(property "Reference" "RN2"
 			(at 137.668 133.2738 0)
 			(show_name no)
@@
 			(project "motherboard-hk10"
 				(path "/e63e39d7-6ac0-4ffd-8aa3-1841a4541b55/00000000-0000-0000-0000-00005ae56078"
-					(reference "RN1")
+					(reference "RN2")
 					(unit 1)
 				)
@@
 		(in_pos_files yes)
 		(dnp no)
-		(property "Reference" "#PWR064"
+		(property "Reference" "#PWR086"
 			(at 132.08 142.24 0)
 			(hide yes)
@@
 			(project "motherboard-hk10"
 				(path "/e63e39d7-6ac0-4ffd-8aa3-1841a4541b55/00000000-0000-0000-0000-00005ae56078"
-					(reference "#PWR064")
+					(reference "#PWR086")
 					(unit 1)
 				)
@@
 		(in_pos_files yes)
 		(dnp no)
-		(property "Reference" "#PWR065"
+		(property "Reference" "#PWR089"
 			(at 146.05 148.59 0)
 			(hide yes)
@@
 			(project "motherboard-hk10"
 				(path "/e63e39d7-6ac0-4ffd-8aa3-1841a4541b55/00000000-0000-0000-0000-00005ae56078"
-					(reference "#PWR065")
+					(reference "#PWR089")
 					(unit 1)
 				)
@@
 		(in_pos_files yes)
 		(dnp no)
-		(property "Reference" "#PWR066"
+		(property "Reference" "#PWR090"
 			(at 146.05 172.72 0)
 			(hide yes)
@@
 			(project "motherboard-hk10"
 				(path "/e63e39d7-6ac0-4ffd-8aa3-1841a4541b55/00000000-0000-0000-0000-00005ae56078"
-					(reference "#PWR066")
+					(reference "#PWR090")
 					(unit 1)
 				)
@@
 		(in_pos_files yes)
 		(dnp no)
-		(property "Reference" "#PWR060"
+		(property "Reference" "#PWR087"
 			(at 139.7 43.18 0)
 			(hide yes)
@@
 			(project "motherboard-hk10"
 				(path "/e63e39d7-6ac0-4ffd-8aa3-1841a4541b55/00000000-0000-0000-0000-00005ae56078"
-					(reference "#PWR060")
+					(reference "#PWR087")
 					(unit 1)
 				)
@@
 		(in_pos_files yes)
 		(dnp no)
-		(property "Reference" "#PWR063"
+		(property "Reference" "#PWR088"
 			(at 139.7 105.41 0)
 			(hide yes)
@@
 			(project "motherboard-hk10"
 				(path "/e63e39d7-6ac0-4ffd-8aa3-1841a4541b55/00000000-0000-0000-0000-00005ae56078"
-					(reference "#PWR063")
+					(reference "#PWR088")
 					(unit 1)
 				)
@@
 		(in_pos_files yes)
 		(dnp no)
-		(property "Reference" "C23"
+		(property "Reference" "C28"
 			(at 146.05 43.18 90)
 			(show_name no)
@@
 			(project "motherboard-hk10"
 				(path "/e63e39d7-6ac0-4ffd-8aa3-1841a4541b55/00000000-0000-0000-0000-00005ae56078"
-					(reference "C23")
+					(reference "C28")
 					(unit 1)
 				)
@@
 		(in_pos_files yes)
 		(dnp no)
-		(property "Reference" "#PWR061"
+		(property "Reference" "#PWR091"
 			(at 153.67 49.53 0)
 			(hide yes)
@@
 			(project "motherboard-hk10"
 				(path "/e63e39d7-6ac0-4ffd-8aa3-1841a4541b55/00000000-0000-0000-0000-00005ae56078"
-					(reference "#PWR061")
-					(unit 1)
-				)
+					(reference "#PWR091")
+					(unit 1)
+				)

Commit message: Adjust footprints and draft PCB layout
Parts:
- C28: footprint PCM_artemisa:Disc_capacitor -> Capacitor_THT:C_Disc_D5.0mm_W2.5mm_P2.50mm
- JP1, JP2, JP3, JP4: footprint PCM_artemisa:Jumper -> Connector_PinHeader_2.54mm:PinHeader_1x03_P2.54mm_Vertical
- RN2: footprint PCM_artemisa:RN4 -> Resistor_THT:R_Array_SIP5
- U21: footprint PCM_artemisa:DIP-32_600 -> Package_DIP:DIP-32_W15.24mm_Socket
Changed lines of the file:
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@@
 			)
 		)
-		(property "Footprint" "PCM_artemisa:DIP-32_600"
+		(property "Footprint" "Package_DIP:DIP-32_W15.24mm_Socket"
 			(at 139.7 69.85 0)
 			(hide yes)
@@
 			)
 		)
-		(property "Footprint" "PCM_artemisa:Jumper"
+		(property "Footprint" "Connector_PinHeader_2.54mm:PinHeader_1x03_P2.54mm_Vertical"
 			(at 110.49 158.75 0)
 			(hide yes)
@@
 			)
 		)
-		(property "Footprint" "PCM_artemisa:Jumper"
+		(property "Footprint" "Connector_PinHeader_2.54mm:PinHeader_1x03_P2.54mm_Vertical"
 			(at 118.11 158.75 0)
 			(hide yes)
@@
 			)
 		)
-		(property "Footprint" "PCM_artemisa:Jumper"
+		(property "Footprint" "Connector_PinHeader_2.54mm:PinHeader_1x03_P2.54mm_Vertical"
 			(at 125.73 158.75 0)
 			(hide yes)
@@
 			)
 		)
-		(property "Footprint" "PCM_artemisa:Jumper"
+		(property "Footprint" "Connector_PinHeader_2.54mm:PinHeader_1x03_P2.54mm_Vertical"
 			(at 133.35 158.75 0)
 			(hide yes)
@@
 			)
 		)
-		(property "Footprint" "PCM_artemisa:RN4"
+		(property "Footprint" "Resistor_THT:R_Array_SIP5"
 			(at 129.54 131.445 0)
 			(hide yes)
@@
 			)
 		)
-		(property "Footprint" "PCM_artemisa:Disc_capacitor"
+		(property "Footprint" "Capacitor_THT:C_Disc_D5.0mm_W2.5mm_P2.50mm"
 			(at 147.32 44.45 0)
 			(hide yes)
