File: slots.kicad_sch (KiCad schematic)
At the start: 6 parts, among them J3 MSX_Slot, J4 MSX_Slot, J5 GFX_Connector_Output, U18 74HCT08

Commit message: Update to KiCad v10 and use plugin-based Artemisa libs
Parts:
- C21: footprint artemisa:Disc_capacitor -> PCM_artemisa:Disc_capacitor; symbol artemisa:Cap -> PCM_artemisa:Cap
- J3, J4: footprint artemisa:Slot_conn -> PCM_artemisa:Slot_conn; symbol artemisa:MSX_Slot -> PCM_artemisa:MSX_Slot
- J5: footprint artemisa:GFX_conn -> PCM_artemisa:GFX_conn; symbol artemisa:GFX_Connector_Output -> PCM_artemisa:GFX_Connector_Output
- RN3: footprint artemisa:RN6 -> PCM_artemisa:RN6; symbol artemisa:RN6 -> PCM_artemisa:RN6
- U18: footprint artemisa:DIP-14_300 -> PCM_artemisa:DIP-14_300; symbol artemisa:74HCT08 -> PCM_artemisa:74HCT08
Connections:
- net ~{EXITINT} renamed ~{EXTINT}
