File: slots.kicad_sch (KiCad schematic)
At the start: 6 parts, among them J3 MSX_Slot, J4 MSX_Slot, J5 GFX_Connector_Output, U18 74HCT08

Commit message: Re-annotate the whole schematic
Parts:
- renumbered C21 to C31, U18 to U24
Changed lines of the file:
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@@
 		(in_pos_files yes)
 		(dnp no)
-		(property "Reference" "#PWR088"
+		(property "Reference" "#PWR0109"
 			(at 328.93 217.17 0)
 			(hide yes)
@@
 			(project "motherboard-hk10"
 				(path "/e63e39d7-6ac0-4ffd-8aa3-1841a4541b55/00000000-0000-0000-0000-00005ae915ed"
-					(reference "#PWR088")
+					(reference "#PWR0109")
 					(unit 1)
 				)
@@
 		(in_pos_files yes)
 		(dnp no)
-		(property "Reference" "#PWR089"
+		(property "Reference" "#PWR0110"
 			(at 334.01 241.3 0)
 			(hide yes)
@@
 			(project "motherboard-hk10"
 				(path "/e63e39d7-6ac0-4ffd-8aa3-1841a4541b55/00000000-0000-0000-0000-00005ae915ed"
-					(reference "#PWR089")
+					(reference "#PWR0110")
 					(unit 1)
 				)
@@
 		(in_pos_files yes)
 		(dnp no)
-		(property "Reference" "#PWR085"
+		(property "Reference" "#PWR0108"
 			(at 266.7 199.39 0)
 			(hide yes)
@@
 			(project "motherboard-hk10"
 				(path "/e63e39d7-6ac0-4ffd-8aa3-1841a4541b55/00000000-0000-0000-0000-00005ae915ed"
-					(reference "#PWR085")
+					(reference "#PWR0108")
 					(unit 1)
 				)
@@
 		(in_pos_files yes)
 		(dnp no)
-		(property "Reference" "#PWR087"
+		(property "Reference" "#PWR0107"
 			(at 233.68 199.39 0)
 			(hide yes)
@@
 			(project "motherboard-hk10"
 				(path "/e63e39d7-6ac0-4ffd-8aa3-1841a4541b55/00000000-0000-0000-0000-00005ae915ed"
-					(reference "#PWR087")
+					(reference "#PWR0107")
 					(unit 1)
 				)
@@
 		(in_pos_files yes)
 		(dnp no)
-		(property "Reference" "#PWR083"
+		(property "Reference" "#PWR0106"
 			(at 228.6 190.5 0)
 			(hide yes)
@@
 			(project "motherboard-hk10"
 				(path "/e63e39d7-6ac0-4ffd-8aa3-1841a4541b55/00000000-0000-0000-0000-00005ae915ed"
-					(reference "#PWR083")
+					(reference "#PWR0106")
 					(unit 1)
 				)
@@
 		(in_pos_files yes)
 		(dnp no)
-		(property "Reference" "#PWR084"
+		(property "Reference" "#PWR0104"
 			(at 179.07 199.39 0)
 			(hide yes)
@@
 			(project "motherboard-hk10"
 				(path "/e63e39d7-6ac0-4ffd-8aa3-1841a4541b55/00000000-0000-0000-0000-00005ae915ed"
-					(reference "#PWR084")
+					(reference "#PWR0104")
 					(unit 1)
 				)
@@
 		(in_pos_files yes)
 		(dnp no)
-		(property "Reference" "#PWR086"
+		(property "Reference" "#PWR0101"
 			(at 146.05 199.39 0)
 			(hide yes)
@@
 			(project "motherboard-hk10"
 				(path "/e63e39d7-6ac0-4ffd-8aa3-1841a4541b55/00000000-0000-0000-0000-00005ae915ed"
-					(reference "#PWR086")
+					(reference "#PWR0101")
 					(unit 1)
 				)
@@
 		(in_pos_files yes)
 		(dnp no)
-		(property "Reference" "#PWR082"
+		(property "Reference" "#PWR099"
 			(at 140.97 190.5 0)
 			(hide yes)
@@
 			(project "motherboard-hk10"
 				(path "/e63e39d7-6ac0-4ffd-8aa3-1841a4541b55/00000000-0000-0000-0000-00005ae915ed"
-					(reference "#PWR082")
+					(reference "#PWR099")
 					(unit 1)
 				)
@@
 		(in_pos_files yes)
 		(dnp no)
-		(property "Reference" "#PWR079"
+		(property "Reference" "#PWR0105"
 			(at 222.25 31.75 0)
 			(hide yes)
@@
 			(project "motherboard-hk10"
 				(path "/e63e39d7-6ac0-4ffd-8aa3-1841a4541b55/00000000-0000-0000-0000-00005ae915ed"
-					(reference "#PWR079")
+					(reference "#PWR0105")
 					(unit 1)
 				)
@@
 		(in_pos_files yes)
 		(dnp no)
-		(property "Reference" "U18"
+		(property "Reference" "U24"
 			(at 176.53 57.15 0)
 			(show_name no)
@@
 			(project "motherboard-hk10"
 				(path "/e63e39d7-6ac0-4ffd-8aa3-1841a4541b55/00000000-0000-0000-0000-00005ae915ed"
-					(reference "U18")
+					(reference "U24")
 					(unit 1)
 				)
@@
 		(in_pos_files yes)
 		(dnp no)
-		(property "Reference" "U18"
+		(property "Reference" "U24"
 			(at 147.32 83.82 0)
 			(show_name no)
@@
 			(project "motherboard-hk10"
 				(path "/e63e39d7-6ac0-4ffd-8aa3-1841a4541b55/00000000-0000-0000-0000-00005ae915ed"
-					(reference "U18")
+					(reference "U24")
 					(unit 2)
 				)
@@
 		(in_pos_files yes)
 		(dnp no)
-		(property "Reference" "U18"
+		(property "Reference" "U24"
 			(at 247.65 73.66 0)
 			(show_name no)
@@
 			(project "motherboard-hk10"
 				(path "/e63e39d7-6ac0-4ffd-8aa3-1841a4541b55/00000000-0000-0000-0000-00005ae915ed"
-					(reference "U18")
+					(reference "U24")
 					(unit 3)
 				)
@@
 		(in_pos_files yes)
 		(dnp no)
-		(property "Reference" "U18"
+		(property "Reference" "U24"
 			(at 220.98 67.31 0)
 			(show_name no)
@@
 			(project "motherboard-hk10"
 				(path "/e63e39d7-6ac0-4ffd-8aa3-1841a4541b55/00000000-0000-0000-0000-00005ae915ed"
-					(reference "U18")
+					(reference "U24")
 					(unit 4)
 				)
@@
 		(in_pos_files yes)
 		(dnp no)
-		(property "Reference" "#PWR081"
+		(property "Reference" "#PWR0111"
 			(at 342.9 107.95 0)
 			(hide yes)
@@
 			(project "motherboard-hk10"
 				(path "/e63e39d7-6ac0-4ffd-8aa3-1841a4541b55/00000000-0000-0000-0000-00005ae915ed"
-					(reference "#PWR081")
+					(reference "#PWR0111")
 					(unit 1)
 				)
@@
 		(in_pos_files yes)
 		(dnp no)
-		(property "Reference" "#PWR0164"
+		(property "Reference" "#PWR0103"
 			(at 172.72 72.39 0)
 			(hide yes)
@@
 			(project "motherboard-hk10"
 				(path "/e63e39d7-6ac0-4ffd-8aa3-1841a4541b55/00000000-0000-0000-0000-00005ae915ed"
-					(reference "#PWR0164")
+					(reference "#PWR0103")
 					(unit 1)
 				)
@@
 		(in_pos_files yes)
 		(dnp no)
-		(property "Reference" "#PWR0165"
+		(property "Reference" "#PWR0102"
 			(at 172.72 45.72 0)
 			(hide yes)
@@
 			(project "motherboard-hk10"
 				(path "/e63e39d7-6ac0-4ffd-8aa3-1841a4541b55/00000000-0000-0000-0000-00005ae915ed"
-					(reference "#PWR0165")
+					(reference "#PWR0102")
 					(unit 1)
 				)
@@
 		(in_pos_files yes)
 		(dnp no)
-		(property "Reference" "C21"
+		(property "Reference" "C31"
 			(at 154.94 46.99 90)
 			(show_name no)
@@
 			(project "motherboard-hk10"
 				(path "/e63e39d7-6ac0-4ffd-8aa3-1841a4541b55/00000000-0000-0000-0000-00005ae915ed"
-					(reference "C21")
+					(reference "C31")
 					(unit 1)
 				)
@@
 		(in_pos_files yes)
 		(dnp no)
-		(property "Reference" "#PWR0178"
+		(property "Reference" "#PWR0100"
 			(at 144.78 57.15 0)
 			(hide yes)
@@
 			(project "motherboard-hk10"
 				(path "/e63e39d7-6ac0-4ffd-8aa3-1841a4541b55/00000000-0000-0000-0000-00005ae915ed"
-					(reference "#PWR0178")
+					(reference "#PWR0100")
 					(unit 1)
 				)

Commit message: Adjust footprints and draft PCB layout
Parts:
- C31: footprint PCM_artemisa:Disc_capacitor -> Capacitor_THT:C_Disc_D5.0mm_W2.5mm_P2.50mm
- J5: footprint PCM_artemisa:GFX_conn -> Connector_IDC:IDC-Header_2x25_P2.54mm_Vertical
- RN3: footprint PCM_artemisa:RN6 -> Resistor_THT:R_Array_SIP7
- U24: footprint PCM_artemisa:DIP-14_300 -> Package_DIP:DIP-14_W7.62mm
Changed lines of the file:
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@@
 			)
 		)
-		(property "Footprint" "PCM_artemisa:GFX_conn"
+		(property "Footprint" "Connector_IDC:IDC-Header_2x25_P2.54mm_Vertical"
 			(at 367.03 146.05 0)
 			(hide yes)
@@
 			)
 		)
-		(property "Footprint" "PCM_artemisa:RN6"
+		(property "Footprint" "Resistor_THT:R_Array_SIP7"
 			(at 219.71 40.005 0)
 			(hide yes)
@@
 			)
 		)
-		(property "Footprint" "PCM_artemisa:DIP-14_300"
+		(property "Footprint" "Package_DIP:DIP-14_W7.62mm"
 			(at 182.88 60.325 0)
 			(hide yes)
@@
 			)
 		)
-		(property "Footprint" "PCM_artemisa:DIP-14_300"
+		(property "Footprint" "Package_DIP:DIP-14_W7.62mm"
 			(at 156.21 80.645 0)
 			(hide yes)
@@
 			)
 		)
-		(property "Footprint" "PCM_artemisa:DIP-14_300"
+		(property "Footprint" "Package_DIP:DIP-14_W7.62mm"
 			(at 256.54 76.835 0)
 			(hide yes)
@@
 			)
 		)
-		(property "Footprint" "PCM_artemisa:DIP-14_300"
+		(property "Footprint" "Package_DIP:DIP-14_W7.62mm"
 			(at 229.87 70.485 0)
 			(hide yes)
@@
 			)
 		)
-		(property "Footprint" "PCM_artemisa:Disc_capacitor"
+		(property "Footprint" "Capacitor_THT:C_Disc_D5.0mm_W2.5mm_P2.50mm"
 			(at 154.94 49.53 0)
 			(hide yes)

Commit message: Connect 12V/-12V rails to slots
Connections:
- net GND: no longer J3.48 (Pin_48), J3.50 (Pin_50), J4.48 (Pin_48), J4.50 (Pin_50), J5.48 (+12V), J5.50 (-12V)
- new net -12V: J3.50 (Pin_50), J4.50 (Pin_50), J5.50 (-12V)
- new net 12V: J3.48 (Pin_48), J4.48 (Pin_48), J5.48 (+12V)
