File: motherboard-hk10.kicad_sch (KiCad schematic)
At the start: 0 parts

Commit message: Introduce PoR using MIC1232
Other:
- sheet Power ports: added CLK; removed none
Changed lines of the file:
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@@
 	)
 	(bus_entry
+		(at 30.48 247.65)
+		(size -2.54 -2.54)
+		(stroke
+			(width 0)
+			(type default)
+		)
+	)
+	(bus_entry
 		(at 30.48 53.34)
 		(size -2.54 2.54)
@@
 	(wire
 		(pts
+			(xy 30.48 247.65) (xy 41.91 247.65)
+		)
+		(stroke
+			(width 0)
+			(type default)
+		)
+	)
+	(wire
+		(pts
 			(xy 41.91 176.53) (xy 30.48 176.53)
 		)
@@
 	(bus
 		(pts
+			(xy 27.94 242.57) (xy 27.94 245.11)
+		)
+		(stroke
+			(width 0)
+			(type default)
+		)
+	)
+	(bus
+		(pts
 			(xy 102.87 97.79) (xy 102.87 119.38)
 		)
@@
 		)
 	)
+	(label "CLK"
+		(at 30.48 247.65 0)
+		(effects
+			(font
+				(size 1.524 1.524)
+			)
+			(justify left bottom)
+		)
+	)
 	(label "~{EXTWAIT}"
 		(at 179.07 125.73 180)
@@
 	(sheet
 		(at 41.91 238.76)
-		(size 29.21 10.16)
+		(size 29.21 12.7)
 		(exclude_from_sim no)
 		(in_bom yes)
@@
 		)
 		(property "Sheetfile" "power.kicad_sch"
-			(at 41.91 249.6062 0)
+			(at 41.91 252.1462 0)
 			(show_name no)
 			(do_not_autoplace no)
@@
 			(effects
 				(font
+					(size 1.524 1.524)
+				)
+				(justify left)
+			)
+		)
+		(pin "CLK" input
+			(at 41.91 247.65 180)
+			(effects
+				(font
