File: motherboard-hk10.kicad_pcb (KiCad board)
At the start: 2 copper layers, 216 x 150 mm, 124 parts, among them J1 PWR_conn, J2 DB25M, J3 MSX_Slot, J4 MSX_Slot, J5 GFX_Connector_Output, J6 CONN_JOY, J7 CONN_JOY, J8 DIN8, K1 Relay, Q1 2N2222, Q2 2N2907, SW1 Push_button, U1 62256, U10 74HC04, U11 74HC32, U12 74HC32, U13 74HC32, U14 74HC08, U15 74HC139, U16 74LS07, U17 74HC74, U18 74HCT08, U19 LM311, U2 62256, U20 SST39SF0, U21 74HC138, U22 74HC138, U23 74HC157, U24 AY-3-8910, U25 74HC157, U26 74HC138, U27 74HC153, U28 82C55A, U3 74HCT244, U4 74HCT244, U5 74HCT244, U6 Z84C00, U7 74HC74, U8 74HCT245, U9 74HCU04, Y1 3.58Mhz

Commit message: Clenaup PCB layout
Parts:
- removed C1, C10, C11, C12, C13, C14, C15, C16, C17, C18, C19, C2, C20, C21, C22, C23, C24, C25, C26, C27, C28, C3, C38, C39, C4, C40, C8, C9: 100nF, artemisa:Disc_capacitor
- removed C29, C30, C31: 10u, artemisa:Radial_capacitor
- removed C32, C35: 1uF, artemisa:Radial_capacitor
- removed C33, C34: 22nF, artemisa:Disc_capacitor
- removed C36, C37: 33pF, artemisa:Disc_capacitor
- removed C5, C7: 100uF, artemisa:Radial_capacitor
- removed C6: 10uF, artemisa:Radial_capacitor
- removed D1, D3: 1N4448, artemisa:Axial_diode
- removed D2: LED, artemisa:LED
- removed G***: LOGO, artemisa:MSX_logo
- removed J1: PWR_conn, artemisa:Jack_55_21
- removed J2: DB25M, artemisa:DB25M
- removed J3, J4: MSX_Slot, artemisa:Slot_conn
- removed J5: GFX_Connector_Output, artemisa:GFX_conn
- removed J6, J7: CONN_JOY, artemisa:Joystick_conn
- removed J8: DIN8, artemisa:DIN8
- removed JP1, JP2, JP3, JP4: Jumper, artemisa:Jumper
- removed K1: Relay, artemisa:Relay
- removed Q1: 2N2222, artemisa:TO92
- removed Q2: 2N2907, artemisa:TO92
- removed R1: 100K, artemisa:Axial_resistor
- removed R10: 20k, artemisa:Axial_resistor
- removed R11, R14, R15, R17: 4k7, artemisa:Axial_resistor
- removed R12, R21, R22: 2k7, artemisa:Axial_resistor
- removed R13: 2k2, artemisa:Axial_resistor
- removed R16: 100, artemisa:Axial_resistor
- removed R18: 220k, artemisa:Axial_resistor
- removed R19: 1k, artemisa:Axial_resistor
- removed R2: 220, artemisa:Axial_resistor
- removed R20: 10k, artemisa:Axial_resistor
- removed R23: 1M, artemisa:Axial_resistor
- removed R24, R5: 1K, artemisa:Axial_resistor
- removed R3, R6: 4K7, artemisa:Axial_resistor
- removed R4, R7, R9: 10K, artemisa:Axial_resistor
- removed R8: 470, artemisa:Axial_resistor
- removed REF** (x6): MountingHole_M3, artemisa:Mounting_hole_M3
- removed RN1, RN5: 10K, artemisa:RN4
- removed RN2, RN4: 10K, artemisa:RN8
- removed RN3: 10K, artemisa:RN6
- removed SW1: Push_button, artemisa:Push_button_angled
- removed U1, U2: 62256, artemisa:DIP-28_600
- removed U10: 74HC04, artemisa:DIP-14_300
- removed U11, U12, U13: 74HC32, artemisa:DIP-14_300
- removed U14: 74HC08, artemisa:DIP-14_300
- removed U15: 74HC139, artemisa:DIP-16_300
- removed U16: 74LS07, artemisa:DIP-14_300
- removed U17, U7: 74HC74, artemisa:DIP-14_300
- removed U18: 74HCT08, artemisa:DIP-14_300
- removed U19: LM311, artemisa:DIP-8_300
- removed U20: SST39SF0, artemisa:DIP-32_600
- removed U21, U22, U26: 74HC138, artemisa:DIP-16_300
- removed U23, U25: 74HC157, artemisa:DIP-16_300
- removed U24: AY-3-8910, artemisa:DIP-40_600
- removed U27: 74HC153, artemisa:DIP-16_300
- removed U28: 82C55A, artemisa:DIP-40_600
- removed U3, U4, U5: 74HCT244, artemisa:DIP-20_300
- removed U6: Z84C00, artemisa:DIP-40_600
- removed U8: 74HCT245, artemisa:DIP-20_300
- removed U9: 74HCU04, artemisa:DIP-14_300
- removed Y1: 3.58Mhz, artemisa:Crystal
Routing:
- net ~: track 1471.7 -> 0.00 mm, vias 20 -> 0
- net /CPU/DATA6: track 595.6 -> 0.00 mm, vias 12 -> 0
- net /CPU/DATA4: track 592.2 -> 0.00 mm, vias 12 -> 0
- net /CPU/DATA3: track 577.3 -> 0.00 mm, vias 10 -> 0
- net /CPU/DATA5: track 576.8 -> 0.00 mm, vias 12 -> 0
- net /CPU/DATA7: track 575.1 -> 0.00 mm, vias 12 -> 0
- net /CPU/DATA2: track 547.7 -> 0.00 mm, vias 10 -> 0
- net /CPU/DATA0: track 539.4 -> 0.00 mm, vias 9 -> 0
- net /~{RESET}: track 535.4 -> 0.00 mm, vias 12 -> 0
- net /CPU/DATA1: track 531.1 -> 0.00 mm, vias 8 -> 0
- net /ADDR1: track 483.7 -> 0.00 mm, vias 11 -> 0
- net /CLK: track 457.2 -> 0.00 mm, vias 11 -> 0
- net /~{RD}: track 456.3 -> 0.00 mm, vias 15 -> 0
- net /ADDR0: track 432.3 -> 0.00 mm, vias 11 -> 0
- net /CPU/ADDR4: track 416.8 -> 0.00 mm, vias 9 -> 0
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- removed copper zone on B.Cu, net GND
- removed copper zone on F.Cu, net GND
Other:
- board outline removed
- board text removed: "Artemisa MSX Computer System Motherboard Model HK-10 - Rev03 Copyright (c) 2018, 2019 Alvaro Polo"
- board text removed: "Cassette connector"
- board text removed: "Graphics card connector"
- board text removed: "JOY A"
- board text removed: "JOY B"
- board text removed: "RESET"
