File: motherboard-hk10.kicad_pcb (KiCad board)
At the start: 2 copper layers, 0 parts

Commit message: Adjust footprints and draft PCB layout
Parts:
- added C1: 100nF, Capacitor_THT:C_Disc_D5.0mm_W2.5mm_P2.50mm, F.Cu at (273.8, 103.1)
- added C10: 100nF, Capacitor_THT:C_Disc_D5.0mm_W2.5mm_P2.50mm, F.Cu at (129.0, 139.3)
- added C11: 100nF, Capacitor_THT:C_Disc_D5.0mm_W2.5mm_P2.50mm, F.Cu at (93.5, 157.1)
- added C12: 100nF, Capacitor_THT:C_Disc_D5.0mm_W2.5mm_P2.50mm, F.Cu at (129.0, 160.9)
- added C13: 100nF, Capacitor_THT:C_Disc_D5.0mm_W2.5mm_P2.50mm, F.Cu at (68.1, 157.8)
- added C14: 100nF, Capacitor_THT:C_Disc_D5.0mm_W2.5mm_P2.50mm, F.Cu at (161.4, 160.9)
- added C15: 100nF, Capacitor_THT:C_Disc_D5.0mm_W2.5mm_P2.50mm, F.Cu at (188.1, 139.3)
- added C16: 100nF, Capacitor_THT:C_Disc_D5.0mm_W2.5mm_P2.50mm, F.Cu at (188.1, 160.9)
- added C17: 100nF, Capacitor_THT:C_Disc_D5.0mm_W2.5mm_P2.50mm, F.Cu at (188.1, 184.4)
- added C18: 100nF, Capacitor_THT:C_Disc_D5.0mm_W2.5mm_P2.50mm, F.Cu at (129.0, 184.4)
- added C19: 100nF, Capacitor_THT:C_Disc_D5.0mm_W2.5mm_P2.50mm, F.Cu at (273.8, 132.3)
- added C2: 100nF, Capacitor_THT:C_Disc_D5.0mm_W2.5mm_P2.50mm, F.Cu at (256.7, 72.7)
- added C20: 100nF, Capacitor_THT:C_Disc_D5.0mm_W2.5mm_P2.50mm, F.Cu at (82.7, 80.9)
- added C21: 10uF, Capacitor_THT:CP_Radial_D4.0mm_P2.00mm, F.Cu at (120.4, 52.3)
- added C22: 100uF, Capacitor_THT:CP_Radial_D5.0mm_P2.50mm, F.Cu at (120.2, 58.1)
- added C23: 10uF, Capacitor_THT:CP_Radial_D4.0mm_P2.00mm, F.Cu at (129.3, 52.3)
- added C24: 100uF, Capacitor_THT:CP_Radial_D5.0mm_P2.50mm, F.Cu at (129.1, 58.1)
- added C25: 10uF, Capacitor_THT:CP_Radial_D4.0mm_P2.00mm, F.Cu at (138.2, 52.3)
- added C26: 100uF, Capacitor_THT:CP_Radial_D5.0mm_P2.50mm, F.Cu at (137.9, 58.1)
- added C27: 100nF, Capacitor_THT:C_Disc_D5.0mm_W2.5mm_P2.50mm, F.Cu at (291.6, 131.1)
- added C28: 100nF, Capacitor_THT:C_Disc_D5.0mm_W2.5mm_P2.50mm, F.Cu at (214.7, 133.0)
- added C29: 100nF, Capacitor_THT:C_Disc_D5.0mm_W2.5mm_P2.50mm, F.Cu at (214.7, 157.1)
- added C3: 100nF, Capacitor_THT:C_Disc_D5.0mm_W2.5mm_P2.50mm, F.Cu at (292.8, 72.6)
- added C30: 100nF, Capacitor_THT:C_Disc_D5.0mm_W2.5mm_P2.50mm, F.Cu at (215.4, 182.5)
- added C31: 100nF, Capacitor_THT:C_Disc_D5.0mm_W2.5mm_P2.50mm, F.Cu at (292.2, 103.1)
- added C32: 10u, Capacitor_THT:CP_Radial_D4.0mm_P2.00mm, F.Cu at (112.5, 130.4)
- added C33: 10u, Capacitor_THT:CP_Radial_D4.0mm_P2.00mm, F.Cu at (163.8, 58.7)
- added C34: 100nF, Capacitor_THT:C_Disc_D5.0mm_W2.5mm_P2.50mm, F.Cu at (68.1, 180.6)
- added C35: 10u, Capacitor_THT:CP_Radial_D4.0mm_P2.00mm, F.Cu at (116.9, 213.6)
- added C36: 100nF, Capacitor_THT:C_Disc_D5.0mm_W2.5mm_P2.50mm, F.Cu at (161.4, 139.3)
- added C37: 100nF, Capacitor_THT:C_Disc_D5.0mm_W2.5mm_P2.50mm, F.Cu at (161.4, 184.4)
- added C38: 1uF, Capacitor_THT:CP_Radial_D4.0mm_P2.00mm, F.Cu at (262.3, 151.4)
- added C39: 22nF, Capacitor_THT:C_Disc_D3.0mm_W2.0mm_P2.50mm, F.Cu at (276.3, 190.8)
- added C4: 100nF, Capacitor_THT:C_Disc_D5.0mm_W2.5mm_P2.50mm, F.Cu at (255.4, 102.5)
- added C40: 100nF, Capacitor_THT:C_Disc_D5.0mm_W2.5mm_P2.50mm, F.Cu at (275.7, 174.3)
- added C41: 22nF, Capacitor_THT:C_Disc_D3.0mm_W2.0mm_P2.50mm, F.Cu at (286.5, 190.8)
- added C42: 1uF, Capacitor_THT:CP_Radial_D4.0mm_P2.00mm, F.Cu at (269.3, 151.4)
- added C5: 100nF, Capacitor_THT:C_Disc_D5.0mm_W2.5mm_P2.50mm, F.Cu at (82.7, 54.9)
- added C6: 100nF, Capacitor_THT:C_Disc_D5.0mm_W2.5mm_P2.50mm, F.Cu at (274.4, 72.6)
- added C7: 100nF, Capacitor_THT:C_Disc_D5.0mm_W2.5mm_P2.50mm, F.Cu at (82.7, 104.4)
- added C8: 100nF, Capacitor_THT:C_Disc_D5.0mm_W2.5mm_P2.50mm, F.Cu at (105.5, 80.9)
- added C9: 100nF, Capacitor_THT:C_Disc_D5.0mm_W2.5mm_P2.50mm, F.Cu at (105.5, 104.4)
- added D1: LED, Connector_PinHeader_2.54mm:PinHeader_1x02_P2.54mm_Vertical, F.Cu at (90.9, 52.5)
- added D2: 1N4448, Diode_THT:D_DO-35_SOD27_P7.62mm_Horizontal, F.Cu at (270.6, 162.8)
- added J1: DB25M, PCM_artemisa:DB25M, F.Cu at (224.1, 226.3)
- added J2: Conn_01x04_Socket, Connector_JST:JST_XH_B4B-XH-A_1x04_P2.50mm_Vertical, F.Cu at (103.0, 52.5)
- added J3: MSX_Slot, PCM_artemisa:Slot_conn, F.Cu at (183.0, 79.1)
- added J4: MSX_Slot, PCM_artemisa:Slot_conn, F.Cu at (182.4, 111.3)
- added J5: GFX_Connector_Output, Connector_IDC:IDC-Header_2x25_P2.54mm_Vertical, F.Cu at (273.8, 55.5)
- added J6: CONN_JOY, PCM_artemisa:Joystick_conn, F.Cu at (94.4, 226.5)
- added J7: CONN_JOY, PCM_artemisa:Joystick_conn, F.Cu at (154.7, 226.5)
- added J8: DIN8, PCM_artemisa:DIN8, F.Cu at (296.0, 160.3)
- added JP1: Jumper, Connector_PinHeader_2.54mm:PinHeader_1x03_P2.54mm_Vertical, F.Cu at (146.8, 52.3)
- added JP2: Jumper, Connector_PinHeader_2.54mm:PinHeader_1x03_P2.54mm_Vertical, F.Cu at (150.6, 52.3)
- added JP3: Jumper, Connector_PinHeader_2.54mm:PinHeader_1x03_P2.54mm_Vertical, F.Cu at (154.4, 52.3)
- added JP4: Jumper, Connector_PinHeader_2.54mm:PinHeader_1x03_P2.54mm_Vertical, F.Cu at (158.2, 52.3)
- added K1: Relay, Relay_THT:Relay_SPDT_Omron-G5LE-1, F.Cu at (274.3, 203.8)
- added Q1: 2N2907, PCM_artemisa:TO92, F.Cu at (263.0, 162.2)
- added R1: 220, Resistor_THT:R_Axial_DIN0207_L6.3mm_D2.5mm_P10.16mm_Horizontal, F.Cu at (90.9, 67.7)
- added R10: 4k7, Resistor_THT:R_Axial_DIN0207_L6.3mm_D2.5mm_P10.16mm_Horizontal, F.Cu at (254.7, 173.6)
- added R11: 2k2, Resistor_THT:R_Axial_DIN0207_L6.3mm_D2.5mm_P10.16mm_Horizontal, F.Cu at (254.7, 177.4)
- added R12: 4k7, Resistor_THT:R_Axial_DIN0207_L6.3mm_D2.5mm_P10.16mm_Horizontal, F.Cu at (254.7, 181.2)
- added R13: 100, Resistor_THT:R_Axial_DIN0207_L6.3mm_D2.5mm_P10.16mm_Horizontal, F.Cu at (254.7, 185.1)
- added R14: 4k7, Resistor_THT:R_Axial_DIN0207_L6.3mm_D2.5mm_P10.16mm_Horizontal, F.Cu at (254.7, 188.9)
- added R15: 220k, Resistor_THT:R_Axial_DIN0207_L6.3mm_D2.5mm_P10.16mm_Horizontal, F.Cu at (254.7, 192.7)
- added R16: 10k, Resistor_THT:R_Axial_DIN0207_L6.3mm_D2.5mm_P10.16mm_Horizontal, F.Cu at (254.7, 196.5)
- added R17: 2k7, Resistor_THT:R_Axial_DIN0207_L6.3mm_D2.5mm_P10.16mm_Horizontal, F.Cu at (254.7, 200.3)
- added R18: 2k7, Resistor_THT:R_Axial_DIN0207_L6.3mm_D2.5mm_P10.16mm_Horizontal, F.Cu at (254.7, 204.1)
- added R2: 4K7, Resistor_THT:R_Axial_DIN0207_L6.3mm_D2.5mm_P10.16mm_Horizontal, F.Cu at (280.8, 145.7)
- added R3: 20k, Resistor_THT:R_Axial_DIN0207_L6.3mm_D2.5mm_P10.16mm_Horizontal, F.Cu at (119.5, 130.4)
- added R4: 4k7, Resistor_THT:R_Axial_DIN0207_L6.3mm_D2.5mm_P10.16mm_Horizontal, F.Cu at (181.7, 52.3)
- added R5: 2k7, Resistor_THT:R_Axial_DIN0207_L6.3mm_D2.5mm_P10.16mm_Horizontal, F.Cu at (127.1, 213.6)
- added R6: 470, Resistor_THT:R_Axial_DIN0207_L6.3mm_D2.5mm_P10.16mm_Horizontal, F.Cu at (68.1, 214.9)
- added R7: 10K, Resistor_THT:R_Axial_DIN0207_L6.3mm_D2.5mm_P10.16mm_Horizontal, F.Cu at (72.5, 204.7)
- added R8: 10K, Resistor_THT:R_Axial_DIN0207_L6.3mm_D2.5mm_P10.16mm_Horizontal, F.Cu at (93.5, 207.3)
- added R9: 1k, Resistor_THT:R_Axial_DIN0207_L6.3mm_D2.5mm_P10.16mm_Horizontal, F.Cu at (291.6, 185.7)
- added RN1: 10K, Resistor_THT:R_Array_SIP9, F.Cu at (230.0, 207.9)
- added RN2: 10K, Resistor_THT:R_Array_SIP5, F.Cu at (163.3, 52.3)
- added RN3: 10K, Resistor_THT:R_Array_SIP7, F.Cu at (282.0, 95.5)
- added RN4: 10K, Resistor_THT:R_Array_SIP9, F.Cu at (172.8, 130.4)
- added RN5: 10K, Resistor_THT:R_Array_SIP5, F.Cu at (170.9, 202.2)
- added SW1: Push_button, PCM_artemisa:Push_button_angled, F.Cu at (266.9, 225.6)
- added U1: 74HC04, Package_DIP:DIP-14_W7.62mm, F.Cu at (263.0, 103.1)
- added U10: 74HC74, Package_DIP:DIP-14_W7.62mm, F.Cu at (94.7, 80.9)
- added U11: 74HCT244, Package_DIP:DIP-20_W7.62mm, F.Cu at (129.0, 150.1)
- added U12: 74HCT244, Package_DIP:DIP-20_W7.62mm, F.Cu at (94.7, 104.4)
- added U13: Z84C00, Package_DIP:DIP-40_W15.24mm_Socket, F.Cu at (68.1, 153.9)
- added U14: 74HCT245, Package_DIP:DIP-20_W7.62mm, F.Cu at (129.0, 171.7)
- added U15: 82C55A, Package_DIP:DIP-40_W15.24mm_Socket, F.Cu at (68.1, 176.2)
- added U16: 74HC153, Package_DIP:DIP-16_W7.62mm, F.Cu at (161.4, 171.7)
- added U17: 74LS07, Package_DIP:DIP-14_W7.62mm, F.Cu at (129.0, 195.2)
- added U18: 74HC138, Package_DIP:DIP-16_W7.62mm, F.Cu at (188.1, 171.7)
- added U19: 74HC138, Package_DIP:DIP-16_W7.62mm, F.Cu at (188.1, 195.2)
- added U2: 74HC32, Package_DIP:DIP-14_W7.62mm, F.Cu at (245.2, 72.7)
- added U20: MIC1232, Package_DIP:DIP-8_W7.62mm, F.Cu at (280.8, 131.1)
- added U21: SST39SF0, Package_DIP:DIP-32_W15.24mm_Socket, F.Cu at (214.7, 151.4)
- added U22: 62256, Package_DIP:DIP-28_W15.24mm_Socket, F.Cu at (214.7, 175.5)
- added U23: 62256, Package_DIP:DIP-28_W15.24mm_Socket, F.Cu at (215.4, 200.9)
- added U24: 74HCT08, Package_DIP:DIP-14_W7.62mm, F.Cu at (281.4, 103.1)
- added U25: AY-3-8910, Package_DIP:DIP-40_W15.24mm_Socket, F.Cu at (68.1, 199.0)
- added U26: 74HC157, Package_DIP:DIP-16_W7.62mm, F.Cu at (161.4, 150.1)
- added U27: 74HC157, Package_DIP:DIP-16_W7.62mm, F.Cu at (161.4, 195.2)
- added U28: LM311, Package_DIP:DIP-8_W7.62mm, F.Cu at (275.7, 185.0)
- added U3: 74HC32, Package_DIP:DIP-14_W7.62mm, F.Cu at (263.6, 72.6)
- added U4: 74HC32, Package_DIP:DIP-14_W7.62mm, F.Cu at (282.1, 72.6)
- added U5: 74HC139, Package_DIP:DIP-16_W7.62mm, F.Cu at (188.1, 150.1)
- added U6: 74HC08, Package_DIP:DIP-14_W7.62mm, F.Cu at (244.6, 102.5)
- added U7: 74HC138, Package_DIP:DIP-16_W7.62mm, F.Cu at (71.9, 54.9)
- added U8: 74HC74, Package_DIP:DIP-14_W7.62mm, F.Cu at (71.9, 80.9)
- added U9: 74HCT244, Package_DIP:DIP-20_W7.62mm, F.Cu at (71.9, 104.4)
- added Y1: SG-531, Oscillator:Oscillator_SeikoEpson_SG-8002DC, F.Cu at (263.0, 132.3)
Other:
- board outline added: 240 x 180 mm
- board text added: "Artemisa Computer System HK-10 Rev01 Copyright(C) 2018-2026 Alvaro Polo"

Commit message: Add mounting holes to the PCB
Parts:
- added H1: MountingHole_3.2mm_M3_DIN965_Pad, MountingHole:MountingHole_3.2mm_M3_DIN965_Pad, F.Cu at (63.9, 55.6)
- added H10: MountingHole_3.2mm_M3_DIN965_Pad, MountingHole:MountingHole_3.2mm_M3_DIN965_Pad, F.Cu at (117.6, 111.4)
- added H11: MountingHole_3.2mm_M3_DIN965_Pad, MountingHole:MountingHole_3.2mm_M3_DIN965_Pad, F.Cu at (237.0, 111.4)
- added H2: MountingHole_3.2mm_M3_DIN965_Pad, MountingHole:MountingHole_3.2mm_M3_DIN965_Pad, F.Cu at (289.9, 55.6)
- added H3: MountingHole_3.2mm_M3_DIN965_Pad, MountingHole:MountingHole_3.2mm_M3_DIN965_Pad, F.Cu at (289.9, 124.6)
- added H4: MountingHole_3.2mm_M3_DIN965_Pad, MountingHole:MountingHole_3.2mm_M3_DIN965_Pad, F.Cu at (289.9, 221.6)
- added H5: MountingHole_3.2mm_M3_DIN965_Pad, MountingHole:MountingHole_3.2mm_M3_DIN965_Pad, F.Cu at (183.9, 221.6)
- added H6: MountingHole_3.2mm_M3_DIN965_Pad, MountingHole:MountingHole_3.2mm_M3_DIN965_Pad, F.Cu at (63.9, 221.6)
- added H7: MountingHole_3.2mm_M3_DIN965_Pad, MountingHole:MountingHole_3.2mm_M3_DIN965_Pad, F.Cu at (63.9, 131.6)
- added H8: MountingHole_3.2mm_M3_DIN965_Pad, MountingHole:MountingHole_3.2mm_M3_DIN965_Pad, F.Cu at (117.6, 79.0)
- added H9: MountingHole_3.2mm_M3_DIN965_Pad, MountingHole:MountingHole_3.2mm_M3_DIN965_Pad, F.Cu at (237.0, 79.0)
- moved C33 30.0 mm to (193.8, 57.4)
- moved R4 12.1 mm to (193.8, 53.0)
- moved RN2 12.1 mm to (175.4, 53.0)
- moved C27 1.28 mm to (292.8, 131.1)
- moved U20 1.28 mm to (282.1, 131.1)
- moved U1 0.90 mm to (263.6, 102.5)
- moved C1 0.90 mm to (274.4, 102.5)
- moved C31 0.90 mm to (292.8, 102.5)
- moved U24 0.90 mm to (282.1, 102.5)
- moved J3 0.65 mm to (182.4, 79.0)
- moved C30 0.65 mm to (214.7, 182.5)
- moved U23 0.64 mm to (214.7, 200.9)
- moved C4 0.64 mm to (256.0, 102.5)
- moved C2 0.63 mm to (256.0, 72.7)
- moved U6 0.63 mm to (245.2, 102.5)
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
Commit message: Fix PCB layout
Parts:
- added H12: MountingHole_3.2mm_M3_DIN965, MountingHole:MountingHole_3.2mm_M3_DIN965, F.Cu at (176.9, 224.6)
- added H13: MountingHole_3.2mm_M3_DIN965, MountingHole:MountingHole_3.2mm_M3_DIN965, F.Cu at (176.9, 52.6)
- added H14: MountingHole_3.2mm_M3_DIN965, MountingHole:MountingHole_3.2mm_M3_DIN965, F.Cu at (60.9, 52.6)
- added H15: MountingHole_3.2mm_M3_DIN965, MountingHole:MountingHole_3.2mm_M3_DIN965, F.Cu at (291.9, 52.6)
- added H16: MountingHole_3.2mm_M3_DIN965, MountingHole:MountingHole_3.2mm_M3_DIN965, F.Cu at (60.9, 224.6)
- added H17: MountingHole_3.2mm_M3_DIN965, MountingHole:MountingHole_3.2mm_M3_DIN965, F.Cu at (292.9, 224.6)
- moved J7 20.8 mm to (133.9, 226.5)
- moved H5 12.2 mm to (176.9, 211.6)
- moved R5 8.72 mm to (120.8, 207.6), turned to 0 degrees
- moved RN2 8.13 mm to (170.3, 59.3)
- moved H1 8.00 mm to (63.9, 63.6)
- moved H2 8.00 mm to (289.9, 63.6)
- moved H4 8.00 mm to (281.9, 221.6)
- moved H6 8.00 mm to (71.9, 221.6)
- moved C35 6.72 mm to (113.9, 207.6)
- moved SW1 6.31 mm to (273.2, 225.6)
- moved J1 5.89 mm to (230.0, 226.3)
- moved C33 4.30 mm to (197.9, 58.7)
Other:
- outline, holes or cut-outs redrawn

Commit message: Connect 12V/-12V rails to slots
Connections:
- J3 pad 48: GND -> 12V
- J3 pad 50: GND -> -12V
- J4 pad 48: GND -> 12V
- J4 pad 50: GND -> -12V
- J5 pad 48: GND -> 12V
- J5 pad 50: GND -> -12V
Changed lines of the file:
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@@
 			(layers "*.Cu" "*.Mask")
 			(remove_unused_layers no)
-			(net "GND")
+			(net "12V")
 			(pinfunction "Pin_48_48")
 			(pintype "passive")
@@
 			(layers "*.Cu" "*.Mask")
 			(remove_unused_layers no)
-			(net "GND")
+			(net "-12V")
 			(pinfunction "Pin_50_50")
 			(pintype "passive")
@@
 			(layers "*.Cu" "*.Mask")
 			(remove_unused_layers no)
-			(net "GND")
+			(net "12V")
 			(pinfunction "Pin_48_48")
 			(pintype "passive")
@@
 			(layers "*.Cu" "*.Mask")
 			(remove_unused_layers no)
-			(net "GND")
+			(net "-12V")
 			(pinfunction "Pin_50_50")
 			(pintype "passive")
@@
 			(layers "*.Cu" "*.Mask")
 			(remove_unused_layers no)
-			(net "GND")
+			(net "12V")
 			(pinfunction "+12V_48")
 			(pintype "power_in")
@@
 			(layers "*.Cu" "*.Mask")
 			(remove_unused_layers no)
-			(net "GND")
+			(net "-12V")
 			(pinfunction "-12V_50")
 			(pintype "power_in")
