File: cassette.kicad_sch (KiCad schematic)
At the start: 20 parts, among them J8 DIN8, K1 Relay, Q2 2N2907, U19 LM311

Commit message: Use clock generator IC instead of oscillator
Parts:
- C22, C33, C34: footprint artemisa:Disc_capacitor -> PCM_artemisa:Disc_capacitor
- C32, C35: footprint artemisa:Radial_capacitor -> PCM_artemisa:Radial_capacitor
- D3: footprint artemisa:Axial_diode -> PCM_artemisa:Axial_diode
- J8: footprint artemisa:DIN8 -> PCM_artemisa:DIN8
- K1: footprint artemisa:Relay -> PCM_artemisa:Relay
- Q2: footprint artemisa:TO92 -> PCM_artemisa:TO92
- R13, R14, R15, R16, R17, R18, R19, R20, R21, R22: footprint artemisa:Axial_resistor -> PCM_artemisa:Axial_resistor; symbol artemisa:R -> PCM_artemisa:R
- U19: footprint artemisa:DIP-8_300 -> PCM_artemisa:DIP-8_300

Commit message: Fix wrong refences to symbols library
Parts:
- C22, C33, C34: symbol artemisa:Cap -> PCM_artemisa:Cap
- C32, C35: symbol artemisa:CP -> PCM_artemisa:CP
- D3: symbol artemisa:1N4448 -> PCM_artemisa:1N4448
- J8: symbol artemisa:DIN8 -> PCM_artemisa:DIN8
- K1: symbol artemisa:Relay -> PCM_artemisa:Relay
- Q2: symbol artemisa:2N2907 -> PCM_artemisa:2N2907
- U19: symbol artemisa:LM311 -> PCM_artemisa:LM311
Changed lines of the file:
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@@
 	)
 	(symbol
-		(lib_id "artemisa:CP")
+		(lib_id "PCM_artemisa:CP")
 		(at 119.38 68.58 90)
 		(unit 1)
@@
 	)
 	(symbol
-		(lib_id "artemisa:Cap")
+		(lib_id "PCM_artemisa:Cap")
 		(at 139.7 73.66 0)
 		(unit 1)
@@
 	)
 	(symbol
-		(lib_id "artemisa:LM311")
+		(lib_id "PCM_artemisa:LM311")
 		(at 139.7 121.92 180)
 		(unit 1)
@@
 	)
 	(symbol
-		(lib_id "artemisa:CP")
+		(lib_id "PCM_artemisa:CP")
 		(at 182.88 138.43 0)
 		(mirror y)
@@
 	)
 	(symbol
-		(lib_id "artemisa:Cap")
+		(lib_id "PCM_artemisa:Cap")
 		(at 171.45 95.25 0)
 		(mirror x)
@@
 	)
 	(symbol
-		(lib_id "artemisa:GND")
+		(lib_id "PCM_artemisa:GND")
 		(at 201.93 90.17 0)
 		(unit 1)
@@
 	)
 	(symbol
-		(lib_id "artemisa:GND")
+		(lib_id "PCM_artemisa:GND")
 		(at 123.19 118.11 0)
 		(unit 1)
@@
 	)
 	(symbol
-		(lib_id "artemisa:GND")
+		(lib_id "PCM_artemisa:GND")
 		(at 182.88 147.32 0)
 		(unit 1)
@@
 	)
 	(symbol
-		(lib_id "artemisa:GND")
+		(lib_id "PCM_artemisa:GND")
 		(at 191.77 147.32 0)
 		(unit 1)
@@
 	)
 	(symbol
-		(lib_id "artemisa:GND")
+		(lib_id "PCM_artemisa:GND")
 		(at 139.7 80.01 0)
 		(unit 1)
@@
 	)
 	(symbol
-		(lib_id "artemisa:GND")
+		(lib_id "PCM_artemisa:GND")
 		(at 157.48 80.01 0)
 		(unit 1)
@@
 	)
 	(symbol
-		(lib_id "artemisa:DIN8")
+		(lib_id "PCM_artemisa:DIN8")
 		(at 217.17 77.47 0)
 		(unit 1)
@@
 	)
 	(symbol
-		(lib_id "artemisa:Relay")
+		(lib_id "PCM_artemisa:Relay")
 		(at 160.02 34.29 0)
 		(unit 1)
@@
 	)
 	(symbol
-		(lib_id "artemisa:1N4448")
+		(lib_id "PCM_artemisa:1N4448")
 		(at 148.59 34.29 90)
 		(unit 1)
@@
 	)
 	(symbol
-		(lib_id "artemisa:GND")
+		(lib_id "PCM_artemisa:GND")
 		(at 151.13 55.88 0)
 		(unit 1)
@@
 	)
 	(symbol
-		(lib_id "artemisa:2N2907")
+		(lib_id "PCM_artemisa:2N2907")
 		(at 151.13 46.99 0)
 		(mirror x)
@@
 	)
 	(symbol
-		(lib_id "artemisa:LM311")
+		(lib_id "PCM_artemisa:LM311")
 		(at 147.32 152.4 0)
 		(unit 2)
@@
 	)
 	(symbol
-		(lib_id "artemisa:GND")
+		(lib_id "PCM_artemisa:GND")
 		(at 139.7 162.56 0)
 		(unit 1)
@@
 	)
 	(symbol
-		(lib_id "artemisa:Cap")
+		(lib_id "PCM_artemisa:Cap")
 		(at 147.32 152.4 0)
 		(unit 1)

Commit message: Re-annotate the whole schematic
Parts:
- renumbered C32 to C38, C33 to C39, C22 to C40, C34 to C41, C35 to C42, D3 to D2, Q2 to Q1, R14 to R10, R13 to R11, R15 to R12, R16 to R13, R17 to R14, R18 to R15, R20 to R16, R21 to R17, R22 to R18, R19 to R9, U19 to U28

Commit message: Adjust footprints and draft PCB layout
Parts:
- C38, C42: footprint PCM_artemisa:Radial_capacitor -> Capacitor_THT:CP_Radial_D4.0mm_P2.00mm
- C39, C41: footprint PCM_artemisa:Disc_capacitor -> Capacitor_THT:C_Disc_D3.0mm_W2.0mm_P2.50mm
- C40: footprint PCM_artemisa:Disc_capacitor -> Capacitor_THT:C_Disc_D5.0mm_W2.5mm_P2.50mm
- D2: footprint PCM_artemisa:Axial_diode -> Diode_THT:D_DO-35_SOD27_P7.62mm_Horizontal
- K1: footprint PCM_artemisa:Relay -> Relay_THT:Relay_SPDT_Omron-G5LE-1
- R10, R11, R12, R13, R14, R15, R16, R17, R18, R9: footprint PCM_artemisa:Axial_resistor -> Resistor_THT:R_Axial_DIN0207_L6.3mm_D2.5mm_P10.16mm_Horizontal
- U28: footprint PCM_artemisa:DIP-8_300 -> Package_DIP:DIP-8_W7.62mm
Changed lines of the file:
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@@
 			)
 		)
-		(property "Footprint" "PCM_artemisa:Radial_capacitor"
+		(property "Footprint" "Capacitor_THT:CP_Radial_D4.0mm_P2.00mm"
 			(at 119.38 68.58 0)
 			(hide yes)
@@
 			)
 		)
-		(property "Footprint" "PCM_artemisa:Axial_resistor"
+		(property "Footprint" "Resistor_THT:R_Axial_DIN0207_L6.3mm_D2.5mm_P10.16mm_Horizontal"
 			(at 130.81 68.58 90)
 			(hide yes)
@@
 			)
 		)
-		(property "Footprint" "PCM_artemisa:Disc_capacitor"
+		(property "Footprint" "Capacitor_THT:C_Disc_D3.0mm_W2.0mm_P2.50mm"
 			(at 139.7 73.66 0)
 			(hide yes)
@@
 			)
 		)
-		(property "Footprint" "PCM_artemisa:Axial_resistor"
+		(property "Footprint" "Resistor_THT:R_Axial_DIN0207_L6.3mm_D2.5mm_P10.16mm_Horizontal"
 			(at 148.59 68.58 90)
 			(hide yes)
@@
 			)
 		)
-		(property "Footprint" "PCM_artemisa:Axial_resistor"
+		(property "Footprint" "Resistor_THT:R_Axial_DIN0207_L6.3mm_D2.5mm_P10.16mm_Horizontal"
 			(at 157.48 73.66 90)
 			(hide yes)
@@
 			)
 		)
-		(property "Footprint" "PCM_artemisa:DIP-8_300"
+		(property "Footprint" "Package_DIP:DIP-8_W7.62mm"
 			(at 139.7 121.92 0)
 			(hide yes)
@@
 			)
 		)
-		(property "Footprint" "PCM_artemisa:Axial_resistor"
+		(property "Footprint" "Resistor_THT:R_Axial_DIN0207_L6.3mm_D2.5mm_P10.16mm_Horizontal"
 			(at 116.84 110.49 90)
 			(hide yes)
@@
 			)
 		)
-		(property "Footprint" "PCM_artemisa:Axial_resistor"
+		(property "Footprint" "Resistor_THT:R_Axial_DIN0207_L6.3mm_D2.5mm_P10.16mm_Horizontal"
 			(at 182.88 121.92 90)
 			(hide yes)
@@
 			)
 		)
-		(property "Footprint" "PCM_artemisa:Radial_capacitor"
+		(property "Footprint" "Capacitor_THT:CP_Radial_D4.0mm_P2.00mm"
 			(at 182.88 138.43 0)
 			(hide yes)
@@
 			)
 		)
-		(property "Footprint" "PCM_artemisa:Axial_resistor"
+		(property "Footprint" "Resistor_THT:R_Axial_DIN0207_L6.3mm_D2.5mm_P10.16mm_Horizontal"
 			(at 191.77 121.92 90)
 			(hide yes)
@@
 			)
 		)
-		(property "Footprint" "PCM_artemisa:Axial_resistor"
+		(property "Footprint" "Resistor_THT:R_Axial_DIN0207_L6.3mm_D2.5mm_P10.16mm_Horizontal"
 			(at 191.77 138.43 90)
 			(hide yes)
@@
 			)
 		)
-		(property "Footprint" "PCM_artemisa:Disc_capacitor"
+		(property "Footprint" "Capacitor_THT:C_Disc_D3.0mm_W2.0mm_P2.50mm"
 			(at 171.45 95.25 0)
 			(hide yes)
@@
 			)
 		)
-		(property "Footprint" "PCM_artemisa:Axial_resistor"
+		(property "Footprint" "Resistor_THT:R_Axial_DIN0207_L6.3mm_D2.5mm_P10.16mm_Horizontal"
 			(at 171.45 106.68 90)
 			(hide yes)
@@
 			)
 		)
-		(property "Footprint" "PCM_artemisa:Axial_resistor"
+		(property "Footprint" "Resistor_THT:R_Axial_DIN0207_L6.3mm_D2.5mm_P10.16mm_Horizontal"
 			(at 182.88 106.68 90)
 			(hide yes)
@@
 			)
 		)
-		(property "Footprint" "PCM_artemisa:Relay"
+		(property "Footprint" "Relay_THT:Relay_SPDT_Omron-G5LE-1"
 			(at 160.655 33.02 0)
 			(hide yes)
@@
 			)
 		)
-		(property "Footprint" "PCM_artemisa:Axial_diode"
+		(property "Footprint" "Diode_THT:D_DO-35_SOD27_P7.62mm_Horizontal"
 			(at 148.59 33.02 0)
 			(hide yes)
@@
 			)
 		)
-		(property "Footprint" "PCM_artemisa:Axial_resistor"
+		(property "Footprint" "Resistor_THT:R_Axial_DIN0207_L6.3mm_D2.5mm_P10.16mm_Horizontal"
 			(at 137.16 46.99 90)
 			(hide yes)
@@
 			)
 		)
-		(property "Footprint" "PCM_artemisa:DIP-8_300"
+		(property "Footprint" "Package_DIP:DIP-8_W7.62mm"
 			(at 147.32 152.4 0)
 			(hide yes)
@@
 			)
 		)
-		(property "Footprint" "PCM_artemisa:Disc_capacitor"
+		(property "Footprint" "Capacitor_THT:C_Disc_D5.0mm_W2.5mm_P2.50mm"
 			(at 147.32 152.4 0)
 			(hide yes)
